File: pcbs/_ready/extend/1.0/_autosave-extend.kicad_pcb (KiCad board)
At the start: 2 copper layers, 85 x 55 mm, 27 parts, among them J1 Conn_01x02_Male, J10 Conn_01x02_Male, J11 Conn_01x02_Pin, J12 Conn_01x03_Pin, J13 Conn_01x02_Male, J14 Conn_01x02_Male, J2 Conn_01x05_Pin, J3 Conn_01x04_Pin, J4 Conn_01x06_Pin, J5 Conn_01x02_Male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

Commit message: Updates
Parts:
- moved J13 0.10 mm to (98.7, 115.1)
- moved J14 0.10 mm to (98.5, 108.7)
- moved J3 0.10 mm to (100.9, 67.0)
- moved J4 0.10 mm to (117.2, 67.0)
- moved J5 0.10 mm to (125.6, 67.0)
- moved J6 0.10 mm to (133.9, 67.0)
- moved J7 0.10 mm to (146.3, 67.0)
- moved J8 0.10 mm to (160.6, 67.0)
Routing:
- net EXPAND: track 0.00 -> 40.6 mm, vias 0 -> 1
Changed lines of the file:
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@@
 	(footprint "Connector_JST:JST_PH_B6B-PH-K_1x06_P2.00mm_Vertical"
 		(layer "F.Cu")
-		(at 117.24 67.1 180)
+		(at 117.24 67 180)
 		(descr "JST PH series connector, B6B-PH-K (http://www.jst-mfg.com/product/pdf/eng/ePH.pdf), generated with kicad-footprint-generator")
 		(tags "connector JST PH side entry")
@@
 	(footprint "Connector_JST:JST_PH_B2B-PH-K_1x02_P2.00mm_Vertical"
 		(layer "F.Cu")
-		(at 98.7 115.2)
+		(at 98.7 115.1)
 		(descr "JST PH series connector, B2B-PH-K (http://www.jst-mfg.com/product/pdf/eng/ePH.pdf), generated with kicad-footprint-generator")
 		(tags "connector JST PH side entry")
@@
 	(footprint "Connector_JST:JST_PH_B5B-PH-K_1x05_P2.00mm_Vertical"
 		(layer "F.Cu")
-		(at 160.6 67.1 180)
+		(at 160.6 67 180)
 		(descr "JST PH series connector, B5B-PH-K (http://www.jst-mfg.com/product/pdf/eng/ePH.pdf), generated with kicad-footprint-generator")
 		(tags "connector JST PH side entry")
@@
 	(footprint "Connector_JST:JST_PH_B4B-PH-K_1x04_P2.00mm_Vertical"
 		(layer "F.Cu")
-		(at 100.9 67.1 180)
+		(at 100.9 67 180)
 		(descr "JST PH series connector, B4B-PH-K (http://www.jst-mfg.com/product/pdf/eng/ePH.pdf), generated with kicad-footprint-generator")
 		(tags "connector JST PH side entry")
@@
 	(footprint "Connector_PinHeader_2.54mm:PinHeader_1x02_P2.54mm_Vertical"
 		(layer "F.Cu")
-		(at 98.56 108.7 90)
+		(at 98.46 108.7 90)
 		(descr "Through hole straight pin header, 1x02, 2.54mm pitch, single row")
 		(tags "Through hole pin header THT 1x02 2.54mm single row")
@@
 	(footprint "Connector_JST:JST_PH_B2B-PH-K_1x02_P2.00mm_Vertical"
 		(layer "F.Cu")
-		(at 125.58 67.1 180)
+		(at 125.58 67 180)
 		(descr "JST PH series connector, B2B-PH-K (http://www.jst-mfg.com/product/pdf/eng/ePH.pdf), generated with kicad-footprint-generator")
 		(tags "connector JST PH side entry")
@@
 	(footprint "Connector_JST:JST_PH_B4B-PH-K_1x04_P2.00mm_Vertical"
 		(layer "F.Cu")
-		(at 146.26 67.1 180)
+		(at 146.26 67 180)
 		(descr "JST PH series connector, B4B-PH-K (http://www.jst-mfg.com/product/pdf/eng/ePH.pdf), generated with kicad-footprint-generator")
 		(tags "connector JST PH side entry")
@@
 	(footprint "Connector_JST:JST_PH_B2B-PH-K_1x02_P2.00mm_Vertical"
 		(layer "F.Cu")
-		(at 133.92 67.1 180)
+		(at 133.92 67 180)
 		(descr "JST PH series connector, B2B-PH-K (http://www.jst-mfg.com/product/pdf/eng/ePH.pdf), generated with kicad-footprint-generator")
 		(tags "connector JST PH side entry")
@@
 	)
 	(segment
+		(start 125.75 96)
+		(end 125.75 97.188096)
+		(width 0.25)
+		(layer "F.Cu")
+		(net 25)
+	)
+	(segment
+		(start 125.75 97.188096)
+		(end 123.938096 99)
+		(width 0.25)
+		(layer "F.Cu")
+		(net 25)
+	)
+	(segment
+		(start 123.938096 99)
+		(end 105.2 99)
+		(width 0.25)
+		(layer "F.Cu")
+		(net 25)
+	)
+	(segment
+		(start 101.1 108.7)
+		(end 101.1 114.8)
+		(width 0.25)
+		(layer "F.Cu")
+		(net 25)
+	)
+	(segment
+		(start 101.1 114.8)
+		(end 100.7 115.2)
+		(width 0.25)
+		(layer "F.Cu")
+		(net 25)
+	)
+	(via
+		(at 105.2 99)
+		(size 0.5)
+		(drill 0.3)
+		(layers "F.Cu" "B.Cu")
+		(net 25)
+	)
+	(segment
+		(start 105.2 99)
+		(end 105.2 104.6)
+		(width 0.25)
+		(layer "B.Cu")
+		(net 25)
+	)
+	(segment
+		(start 105.2 104.6)
+		(end 101.1 108.7)
+		(width 0.25)
+		(layer "B.Cu")
+		(net 25)
+	)
+	(segment
