File: pcbs/mono/1.0/mono.kicad_pcb (KiCad board)
At the start: 2 copper layers, 100 x 45 mm, 39 parts, among them J1 Conn_01x03_Pin, J10 Conn_01x02_Pin, J11 Conn_01x02_Pin, J2 Conn_01x03_Male, J3 Conn_01x03_Pin, J4 Conn_01x02_Pin, J5 Conn_01x04_Pin, J6 Conn_01x03_Male, J7 Conn_01x03_Male, J8 Conn_01x02_Pin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

Commit message: Major updates
Changed lines of the file:
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@@
 	(segment
 		(start 127.8175 77.64375)
-		(end 129.4 79.22625)
+		(end 127.7 77.76125)
 		(width 2.5)
 		(layer "F.Cu")
@@
 	)
 	(segment
-		(start 129.4 79.22625)
+		(start 129.4 83)
 		(end 129.4 87.5)
 		(width 2.5)
 		(layer "F.Cu")
+		(net 2)
+	)
+	(segment
+		(start 127.7 81.3)
+		(end 129.4 83)
+		(width 2.5)
+		(layer "F.Cu")
+		(net 2)
+	)
+	(segment
+		(start 127.7 77.76125)
+		(end 127.7 81.3)
+		(width 2.5)
+		(layer "F.Cu")
