File: pcbs/plate-amp/1.0/plate-amp.kicad_sch (KiCad schematic)
At the start: 32 parts, among them J1 Conn_01x02_Pin, J2 Conn_01x02_Pin, J3 Conn_01x02_Pin, U1 TPA3255DDV, U3 OPA1602, U4 OPA1602

Commit message: Major updates
Parts:
- removed C11, C12: 10n C0G, Capacitor_SMD:C_1206_3216Metric, symbol Device:C_Small
- removed C17: 33n C0G, Capacitor_SMD:C_0805_2012Metric, symbol Device:C_Small
- added C11, C12, C17, C18: 1000U 50V, Capacitor_THT:CP_Radial_D12.5mm_P5.00mm, symbol Device:C_Polarized_Small
- added C19, C20: 1U X7R 50V, Capacitor_SMD:C_1206_3216Metric_Pad1.33x1.80mm_HandSolder, symbol Device:C_Polarized_Small
- added C21, C22, C23, C24: 33n 100V, Capacitor_SMD:C_1206_3216Metric_Pad1.33x1.80mm_HandSolder, symbol Device:C_Small
- added C25, C30, C31, C32: 0.1u, Capacitor_SMD:C_0805_2012Metric_Pad1.18x1.45mm_HandSolder, symbol Device:C_Small
- added C26, C27, C28, C29, C37, C39: 10u Nichicon 25V, Capacitor_THT:CP_Radial_D5.0mm_P2.50mm, symbol Device:C_Small
- added C33, C34, C35: 1u, Capacitor_SMD:C_1206_3216Metric_Pad1.33x1.80mm_HandSolder, symbol Device:C_Small
- added C36, C41, C42: 10u 50V, Capacitor_SMD:C_1206_3216Metric_Pad1.33x1.80mm_HandSolder, symbol Device:C_Small
- added C38, C43: 47u, Capacitor_SMD:C_1206_3216Metric_Pad1.33x1.80mm_HandSolder, symbol Device:C_Small
- added C40: 470u 16V, Capacitor_THT:CP_Radial_D8.0mm_P3.50mm, symbol Device:C_Small
- added D2: RED, LED_SMD:LED_0603_1608Metric_Pad1.05x0.95mm_HandSolder, symbol Device:LED
- added H3, H4: MountingHole_Pad, MountingHole:MountingHole_3.2mm_M3_DIN965_Pad_TopBottom, symbol Mechanical:MountingHole_Pad
- added J3: Conn_01x02_Pin, Connector_JST:JST_VH_B2P-VH-B_1x02_P3.96mm_Vertical, symbol Connector:Conn_01x02_Pin
- added J4, J8: Conn_01x02_Pin, Connector_JST:JST_PH_B2B-PH-K_1x02_P2.00mm_Vertical, symbol Connector:Conn_01x02_Pin
- added J5: Conn_01x03_Pin, Connector_JST:JST_PH_B3B-PH-K_1x03_P2.00mm_Vertical, symbol Connector:Conn_01x03_Pin
- added J6: Conn_01x04_Pin, Connector_JST:JST_PH_B4B-PH-K_1x04_P2.00mm_Vertical, symbol Connector:Conn_01x04_Pin
- added R10: 30k, Capacitor_SMD:C_0603_1608Metric_Pad1.08x0.95mm_HandSolder, symbol Device:R_Small
- added R11, R8: 3R3, Capacitor_SMD:C_0603_1608Metric_Pad1.08x0.95mm_HandSolder, symbol Device:R_Small
- added R12, R14, R15, R16, R18, R25, R26, R27: 10k, Capacitor_SMD:C_0603_1608Metric_Pad1.08x0.95mm_HandSolder, symbol Device:R_Small
- added R13, R17, R20, R21, R23, R24: 20k, Capacitor_SMD:C_0603_1608Metric_Pad1.08x0.95mm_HandSolder, symbol Device:R_Small
- added R19, R22: 13k, Capacitor_SMD:C_0603_1608Metric_Pad1.08x0.95mm_HandSolder, symbol Device:R_Small
- added R3, R4: 3R3, Resistor_SMD:R_2512_6332Metric_Pad1.40x3.35mm_HandSolder, symbol Device:R_Small
- added R6: 330R, Resistor_SMD:R_0603_1608Metric_Pad0.98x0.95mm_HandSolder, symbol Device:R_Small
- added R7: 4.7K, Resistor_SMD:R_0603_1608Metric_Pad0.98x0.95mm_HandSolder, symbol Device:R_Small
- added R9: 22k, Capacitor_SMD:C_0603_1608Metric_Pad1.08x0.95mm_HandSolder, symbol Device:R_Small
- added U2: ~, Custom:UA8014-AL, symbol Custom:UA8014-AL
- added U3: TMP100, Package_TO_SOT_SMD:SOT-23-6, symbol Sensor_Temperature:TMP100
- C1, C2: value 1000u 63V -> 47U 50V; footprint Capacitor_THT:CP_Radial_D16.0mm_P7.50mm -> Capacitor_THT:CP_Radial_D6.3mm_P2.50mm
- C10, C9: value 1n C0G -> 10n 50V C0G; footprint Capacitor_SMD:C_1206_3216Metric -> Capacitor_SMD:C_1206_3216Metric_Pad1.33x1.80mm_HandSolder
- C13: value 10u Nichicon 25V -> 1u 50V; footprint Capacitor_THT:CP_Radial_D5.0mm_P2.50mm -> Capacitor_THT:CP_Radial_D5.0mm_P2.00mm
- C14, C15, C16: value 33n C0G -> 1u 50V; footprint Capacitor_SMD:C_0805_2012Metric -> Capacitor_THT:CP_Radial_D5.0mm_P2.00mm
- C3, C4: value 10u Nichicon 25V -> 1n 50V C0G; footprint Capacitor_THT:CP_Radial_D5.0mm_P2.50mm -> Capacitor_SMD:C_1206_3216Metric_Pad1.33x1.80mm_HandSolder
- C5, C6: value 470n 100V -> 1n 50V C0G; footprint Capacitor_THT:C_Rect_L18.0mm_W9.0mm_P15.00mm_FKS3_FKP3 -> Capacitor_SMD:C_1206_3216Metric_Pad1.33x1.80mm_HandSolder
- C7, C8: value 470n 100V -> 10n 50V C0G; footprint Capacitor_THT:C_Rect_L18.0mm_W9.0mm_P15.00mm_FKS3_FKP3 -> Capacitor_SMD:C_1206_3216Metric_Pad1.33x1.80mm_HandSolder
- R1, R2: footprint Resistor_SMD:R_2010_5025Metric_Pad1.40x2.65mm_HandSolder -> Resistor_SMD:R_2512_6332Metric_Pad1.40x3.35mm_HandSolder
- R5: value 150R -> 3K
- renumbered D3 to D1, H4 to H1, H3 to H2, H2 to H5, H1 to H6, J2 to J1, J1 to J2, J3 to J7, U2 to U1, U1 to U4, U3 to U5, U4 to U6
Connections:
- net GND1 is gone; now on net PGND: U4.41 (GND), U4.42 (GND)
- net GND2 is gone; now on net PGND: U4.25 (GND), U4.26 (GND)
- net GNDMID is gone; now on net PGND: U4.33 (GND), U4.34 (GND)
- net INA is gone; now on net SPEAKERL_POS: C3.1
- net INB is gone; now on net PGND: C4.1
- net 12V: now also R5.1, U4.2 (VDD), C31.2, C40.1, J6.4 (Pin_4), R11.1, R8.1; no longer U5.8 (V+), U6.8 (V+)
- net 3V3: now also C25.2, C36.1, J6.2 (Pin_2), U3.3 (ADD1), U3.4 (V+); no longer R5.1
- net 48V: now also C11.1, C12.1, C17.1, C18.1, C19.1, C20.1
- net GND: now also U4.3 (M1), U4.4 (M2), C25.1, C30.2, C31.1, C32.2, C33.1, C34.1, C35.1, C36.2, C38.2, C40.2, C41.2, C42.2, C43.1, D2.1 (K), J6.1 (Pin_1), J8.1 (Pin_1), R10.1, R13.1, R17.1, R21.1, R23.1, R25.1, R7.2, R9.1, U3.2 (GND), U3.5 (ADD0); no longer C1.2, C2.2, J2.1 (Pin_1), U4.45 (EP)
- net 4.75V: now reaches U5.5 (+)
- net 4.75V: now also U5.3 (+), U6.3 (+), U6.5 (+), C38.1, R12.1, R20.2, R24.2, R25.2
- net at U5.6 (-): now also R14.2, R15.1
- net at U5.7: now also C27.2, R14.1
- net LEFT_B: now reaches U4.6 (INPUT_B)
- net LEFT_B: now also C27.1, R13.2; no longer C4.2
- net at U4.43 (BST_B): now also C21.1
- net PGND: now reaches R2.1
- net PGND: now also C1.2, C13.2, C14.1, C15.2, C16.1, C2.2, C3.2, C5.2, C6.1, J2.1 (Pin_1), R1.2, U4.45 (EP), C11.2, C12.2, C17.2, C18.2, C19.2, C20.2, H3.1, H4.1, R3.2, R4.1
- net at U4.44 (BST_A): now also C23.1; no longer C16.2
- net at U5.1: now also C26.2, R15.2, R19.1
- net at U5.2 (-): now also R19.2, R27.1
- net SPEAKERL_POS: now reaches C13.1
- net SPEAKERL_POS: now also C7.1, J1.1 (Pin_1), U1.3 (L2_OUT); no longer U5.3 (+)
- net at U4.24 (BST_C): now also C22.1; no longer C14.2
- net at U4.23 (BST_D): now also C24.1; no longer C15.2
- net LEFT_A: now reaches U4.5 (INPUT_A)
- net LEFT_A: now also C26.1, R21.2; no longer C3.2
- net at U6.6 (-): now also R16.2, R18.1
- net at U6.7: now also C29.2, R16.1
- net at U6.1: now also C28.2, R18.2, R22.1
- net at U6.2 (-): now also R22.2, R26.1
- net at U4.1 (GVDD_AB): now also C30.1, R8.2
- net at U4.11 (DVDD): now also C33.2
- net at U4.14 (AVDD): now also C34.2
- net at U4.15 (C_START): now also C43.2
- net RIGHT_A: now reaches U4.16 (INPUT_C)
- net RIGHT_A: now also C28.1, R23.2
- net RIGHT_B: now reaches U4.17 (INPUT_D)
- net RIGHT_B: now also C29.1, R17.2
- net RESET: now reaches U4.18 (~{RESET})
- net RESET: now also J5.1 (Pin_1), R6.1, R7.1
- net FAULT: now reaches U4.19 (~{FAULT})
- net FAULT: now also J5.2 (Pin_2)
- net at U4.20 (VBG): now also C35.2
- net CLIP: now reaches U4.21 (~{CLIP_OTW})
- net CLIP: now also J5.3 (Pin_3)
- net at U4.22 (GVDD_CD): now also C32.1, R11.2
- net at U4.7 (OC_ADJ): now also R9.2
- net at U4.8 (FREQ_ADJ): now also R10.2
- net AUDIO_IN renamed LEFT_IN
- net LEFT_IN: now also C37.2; no longer C13.2
- removed net MID: C10.2, C5.1, C6.2, C7.1, C8.2, C9.1, R1.1, R2.2
- net OUT1 renamed OUTA
- net OUTA: now also C23.2; no longer C14.1, C16.1, U4.32 (OUT_C)
- removed net OUT2: C15.1, U1.1 (L1_IN), U4.27 (OUT_D), U4.28 (OUT_D), U4.35 (OUT_B)
- removed net SPEAKER_OUT1: C5.2, C7.2, C9.2, J1.1 (Pin_1), U1.3 (L2_OUT)
- removed net SPEAKER_OUT2: C10.1, C6.1, C8.1, J1.2 (Pin_2), U1.2 (L1_OUT)
- new net: C9.2, R3.1
- new net: C7.2, R1.1
- new net: C37.1, R20.1, R27.2
- new net: C10.1, R4.2
- new net: D2.2 (A), R6.2
- new net: C39.1, R24.1, R26.2
- new net: C8.1, R2.2
- new net 9.5V: C41.1, C42.1, J6.3 (Pin_3), R12.2, U5.8 (V+), U6.8 (V+)
- new net OUTB: C21.2, U1.1 (L1_IN), U4.35 (OUT_B)
- new net OUTC: C22.2, U2.4 (L2_IN), U4.32 (OUT_C)
- new net OUTD: C24.2, U2.1 (L1_IN), U4.27 (OUT_D), U4.28 (OUT_D)
- new net RIGHT_IN: C39.2, J8.2 (Pin_2)
- new net SCL: J4.1 (Pin_1), U3.1 (SCL)
- new net SDA: J4.2 (Pin_2), U3.6 (SDA)
- new net SPEAKERL_NEG: C14.2, C4.2, C8.2, J1.2 (Pin_2), U1.2 (L1_OUT)
- new net SPEAKERR_NEG: C10.2, C16.2, C6.2, J3.2 (Pin_2), U2.2 (L1_OUT)
- new net SPEAKERR_POS: C15.1, C5.1, C9.1, J3.1 (Pin_1), U2.3 (L2_OUT)
Other:
- moved on the sheet: D1, R5, U1, U4, U5A, U5B, U5C, U6A, U6B, U6C
