File: pcbs/adc/1.1/adc.kicad_pcb (KiCad board)
At the start: 2 copper layers, 85 x 55 mm, 51 parts, among them J1 Conn_01x04_Pin, J2 Conn_01x02_Male, J3 Conn_01x03_Pin, J4 Conn_01x04_Pin, J5 Conn_01x03_Pin, J6 Conn_01x03_Pin, U1 ASDMB-xxxMHz, U2 ZLDO1117QG33TA, U3 PCM1863

Commit message: Updates
Parts:
- moved C12 7.64 mm to (150.6, 88.6), turned to 180 degrees
- moved D3 5.55 mm to (152.3, 69.3)
- moved D1 5.55 mm to (152.3, 63.5)
- moved D2 5.55 mm to (152.3, 66.4)
- moved R1 5.55 mm to (149.0, 63.5)
- moved R2 5.55 mm to (149.0, 66.4)
- moved R4 5.55 mm to (149.0, 69.3)
- moved U2 4.99 mm to (152.5, 82.2)
- moved C3 2.32 mm to (150.6, 75.9), turned to 180 degrees
- moved J2 1.02 mm to (162.0, 105.1)
- moved C13 0.14 mm to (120.0, 89.4)
- moved C11 0.06 mm to (119.4, 86.0)
- moved C9 0.06 mm to (118.8, 83.6)
- renumbered C11 to C10, C12 to C11, C9 to C12, C10 to C9, R9 to R10, R10 to R11, R11 to R12, R12 to R3, R3 to R4, R4 to R5, R5 to R6, R6 to R7, R7 to R8, R8 to R9
Routing:
- net 3V3A: track 79.9 -> 92.0 mm, vias 2 -> 4
- net GND: track 35.4 -> 39.5 mm
- net 5V: track 49.8 -> 46.6 mm, vias 2 -> 0
- net ADC_INT: track 28.2 -> 29.2 mm
- net Net-(C20-Pad2): track 8.80 -> 9.74 mm
- net SDA: track 27.0 -> 27.8 mm
- net Net-(C21-Pad2): track 7.94 -> 8.67 mm
- net 3V3: track 128.9 -> 129.7 mm
Other:
- board text added: "ADC 1.1"
- board text removed: "ADC 1.0"
