File: pcbs/adc/1.1/adc.kicad_sch (KiCad schematic)
At the start: 51 parts, among them J1 Conn_01x04_Pin, J2 Conn_01x02_Male, J3 Conn_01x03_Pin, J4 Conn_01x04_Pin, J5 Conn_01x03_Pin, J6 Conn_01x03_Pin, U1 ASDMB-xxxMHz, U2 ZLDO1117QG33TA, U3 PCM1863

Commit message: Updates
Parts:
- renumbered C11 to C10, C12 to C11, C9 to C12, C10 to C9, R9 to R10, R10 to R11, R11 to R12, R12 to R3, R3 to R4, R4 to R5, R5 to R6, R6 to R7, R7 to R8, R8 to R9
Changed lines of the file:
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@@
 		(dnp no)
 		(fields_autoplaced yes)
-		(property "Reference" "R5"
+		(property "Reference" "R6"
 			(at 299.72 107.95 90)
 			(effects
@@
 			(project "ADC"
 				(path "/ad933f83-dd94-4dcc-b4f2-96fd54138c43"
-					(reference "R5")
+					(reference "R6")
 					(unit 1)
 				)
@@
 		(dnp no)
 		(fields_autoplaced yes)
-		(property "Reference" "R6"
+		(property "Reference" "R7"
 			(at 292.1 110.49 90)
 			(effects
@@
 			(project "ADC"
 				(path "/ad933f83-dd94-4dcc-b4f2-96fd54138c43"
-					(reference "R6")
+					(reference "R7")
 					(unit 1)
 				)
@@
 		(on_board yes)
 		(dnp no)
-		(property "Reference" "R12"
+		(property "Reference" "R3"
 			(at 69.342 114.3 0)
 			(effects
@@
 			(project "adc"
 				(path "/ad933f83-dd94-4dcc-b4f2-96fd54138c43"
-					(reference "R12")
+					(reference "R3")
 					(unit 1)
 				)
@@
 		(dnp no)
 		(fields_autoplaced yes)
-		(property "Reference" "C11"
+		(property "Reference" "C10"
 			(at 162.814 37.2999 0)
 			(effects
@@
 			(project "ChannelSelector"
 				(path "/ad933f83-dd94-4dcc-b4f2-96fd54138c43"
-					(reference "C11")
+					(reference "C10")
 					(unit 1)
 				)
@@
 		(dnp no)
 		(fields_autoplaced yes)
-		(property "Reference" "R8"
+		(property "Reference" "R9"
 			(at 194.31 116.84 90)
 			(effects
@@
 			(project "adc"
 				(path "/ad933f83-dd94-4dcc-b4f2-96fd54138c43"
-					(reference "R8")
+					(reference "R9")
 					(unit 1)
 				)
@@
 		(dnp no)
 		(fields_autoplaced yes)
-		(property "Reference" "R11"
+		(property "Reference" "R12"
 			(at 147.32 100.33 90)
 			(effects
@@
 			(project "ADC"
 				(path "/ad933f83-dd94-4dcc-b4f2-96fd54138c43"
-					(reference "R11")
+					(reference "R12")
 					(unit 1)
 				)
@@
 		(dnp no)
 		(fields_autoplaced yes)
-		(property "Reference" "R3"
+		(property "Reference" "R4"
 			(at 109.22 29.2099 0)
 			(effects
@@
 			(project "ADC"
 				(path "/ad933f83-dd94-4dcc-b4f2-96fd54138c43"
-					(reference "R3")
+					(reference "R4")
 					(unit 1)
 				)
@@
 		(dnp no)
 		(fields_autoplaced yes)
-		(property "Reference" "R9"
+		(property "Reference" "R10"
 			(at 194.31 124.46 90)
 			(effects
@@
 			(project "adc"
 				(path "/ad933f83-dd94-4dcc-b4f2-96fd54138c43"
-					(reference "R9")
+					(reference "R10")
 					(unit 1)
 				)
@@
 		(dnp no)
 		(fields_autoplaced yes)
-		(property "Reference" "R4"
+		(property "Reference" "R5"
 			(at 292.1 127 90)
 			(effects
@@
 			(project "ADC"
 				(path "/ad933f83-dd94-4dcc-b4f2-96fd54138c43"
-					(reference "R4")
+					(reference "R5")
 					(unit 1)
 				)
@@
 		(dnp no)
 		(fields_autoplaced yes)
-		(property "Reference" "C10"
+		(property "Reference" "C9"
 			(at 226.06 41.9162 0)
 			(effects
@@
 			(project "ADC"
 				(path "/ad933f83-dd94-4dcc-b4f2-96fd54138c43"
-					(reference "C10")
+					(reference "C9")
 					(unit 1)
 				)
@@
 		(dnp no)
 		(fields_autoplaced yes)
-		(property "Reference" "C12"
+		(property "Reference" "C11"
 			(at 236.22 41.9162 0)
 			(effects
@@
 			(project "ADC"
 				(path "/ad933f83-dd94-4dcc-b4f2-96fd54138c43"
-					(reference "C12")
+					(reference "C11")
 					(unit 1)
 				)
@@
 		(dnp no)
 		(fields_autoplaced yes)
-		(property "Reference" "R10"
+		(property "Reference" "R11"
 			(at 147.32 92.71 90)
 			(effects
@@
 			(project "ADC"
 				(path "/ad933f83-dd94-4dcc-b4f2-96fd54138c43"
-					(reference "R10")
+					(reference "R11")
 					(unit 1)
 				)
@@
 		(dnp no)
 		(fields_autoplaced yes)
-		(property "Reference" "R7"
+		(property "Reference" "R8"
 			(at 285.75 113.03 90)
 			(effects
@@
 			(project "ADC"
 				(path "/ad933f83-dd94-4dcc-b4f2-96fd54138c43"
-					(reference "R7")
+					(reference "R8")
 					(unit 1)
 				)
@@
 		(on_board yes)
 		(dnp no)
-		(property "Reference" "C9"
+		(property "Reference" "C12"
 			(at 58.801 111.7536 0)
 			(effects
@@
 			(project "ADC"
 				(path "/ad933f83-dd94-4dcc-b4f2-96fd54138c43"
-					(reference "C9")
+					(reference "C12")
 					(unit 1)
 				)
