File: pcbs/dolby/1.2 Draft/dsp.kicad_sch (KiCad schematic)
At the start: 74 parts, among them J1 Conn_01x04_Pin, J2 Conn_01x04_Pin, J3 Conn_01x02, J4 Conn_01x02_Pin, J5 Conn_01x03_Pin, J6 Conn_01x04_Male, J7 Conn_01x02, U1 TLV1117LV-25, U2 AZ1117CH2-3.3, U3 DA101C_C6931652, U4 SPA130, U5 TLV1117LV-25, U6 TMP100, X1 ECS-3225SMV-270-FP-TR

Commit message: UPdates
Parts:
- removed C11: 10U, Capacitor_SMD:C_1206_3216Metric_Pad1.33x1.80mm_HandSolder, symbol Device:C_Small
- removed U2: AZ1117CH2-3.3, Package_TO_SOT_SMD:SOT-223-3_TabPin2, symbol Regulator_Linear:AMS1117-2.5
- removed U6: TMP100, Package_TO_SOT_SMD:SOT-23-6, symbol Sensor_Temperature:TMP100
- added C17, C6: 10U, Capacitor_SMD:C_1206_3216Metric_Pad1.33x1.80mm_HandSolder, symbol Device:C_Small
- added C2: 220u, Capacitor_THT:CP_Radial_D6.3mm_P2.50mm, symbol Device:C_Polarized
- added C20: 0.1U, Capacitor_SMD:C_0805_2012Metric_Pad1.18x1.45mm_HandSolder, symbol Device:C_Small
- added J8: Conn_01x02, Connector_PinHeader_2.54mm:PinHeader_1x02_P2.54mm_Vertical, symbol Connector_Generic:Conn_01x02
- added J9: Conn_01x04_Pin, Connector_PinHeader_2.54mm:PinHeader_1x04_P2.54mm_Vertical, symbol Connector:Conn_01x04_Pin
- added TP1, TP2, TP3: TestPoint, TestPoint:TestPoint_THTPad_1.5x1.5mm_Drill0.7mm, symbol Connector:TestPoint
- added U4: AZ1117CH2-3.3, Package_TO_SOT_SMD:SOT-223-3_TabPin2, symbol Regulator_Linear:AMS1117-2.5
- C16: value 0.1U -> 10U; footprint Capacitor_SMD:C_0805_2012Metric_Pad1.18x1.45mm_HandSolder -> Capacitor_SMD:C_1206_3216Metric_Pad1.33x1.80mm_HandSolder
- renumbered C5 to C10, C6 to C11, C8 to C12, C7 to C13, C9 to C14, C12 to C15, C14 to C18, C15 to C19, C20 to C21, C21 to C22, C13 to C23, C22 to C24, C17 to C25, C24 to C26, C25 to C27, C26 to C28, C27 to C29, C10 to C3, C28 to C31, C29 to C32, C31 to C33, C23 to C34, C32 to C36, C33 to C37, C18 to C4, C2 to C5, C19 to C7, C3 to C8, C4 to C9, J4 to J3, J3 to J4, R7 to R6, R8 to R7, R6 to R8, U5 to U2, U4 to U5
Connections:
- net 3V3A is gone; now on net 2.5V: C1.1
- net SPDIF_NEG is gone; now on net AGND: C25.1, R8.2, U3.4
- net 2.5V: now also TP3.1
- net 3V3: now also C6.1; no longer C10.1, C12.1, C16.2, C19.1, C33.1, C36.1, C8.1, R10.2, R19.1, R6.1, R9.1, U5.10 (VDD3), U5.32 (VDD3), U5.51 (VDD3), U5.70 (VDD3), X1.1 (EN), X1.4 (Vdd)
- net 5V: now also C16.1, U4.3 (VI)
- net AGND: now also C16.2, C17.2, C6.2, TP2.1, U4.1 (GND)
- net BCLK: now also J9.2 (Pin_2)
- net GND: now also C2.2, C20.2, J8.1 (Pin_1), TP1.1; no longer C16.1, J5.2 (Pin_2)
- net I2S_D1: now also J9.4 (Pin_4)
- net PCMCLK: now also J9.1 (Pin_1)
- net WCLK: now also J9.3 (Pin_3)
- net at R1.1: now also U5.76 (PCM_OUT2); no longer U5.77 (PCM_OUT3)
- new net 3V3_2: C10.1, C12.1, C17.1, C19.1, C2.1, C20.1, C33.1, C36.1, C8.1, R10.2, R19.1, R6.1, R9.1, U4.2 (VO), U5.10 (VDD3), U5.32 (VDD3), U5.51 (VDD3), U5.70 (VDD3), X1.1 (EN), X1.4 (Vdd)
- new net GND_IN: J5.2 (Pin_2), J8.2 (Pin_2)
Other:
- moved on the sheet: R1
