File: pcbs/psu-multi/1.0/multipsu.kicad_sch (KiCad schematic)
At the start: 61 parts, among them J1 Conn_01x06_Pin, J2 Conn_01x03_Male, J3 Conn_01x02_Pin, J4 Conn_01x02_Pin, J5 Conn_01x03_Pin, J6 Conn_01x03_Pin, U1 LM337_SOT223, U10 INA260, U11 INA260, U12 INA260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

Commit message: UPdates
Changed lines of the file:
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@@
 (kicad_sch
-	(version 20231120)
+	(version 20250114)
 	(generator "eeschema")
-	(generator_version "8.0")
+	(generator_version "9.0")
 	(paper "A2")
 	(junction
@@
 		)
 	)
+	(embedded_fonts no)
 )
