File: pcbs/dsp/1.2 Draft/dsp.kicad_sch (KiCad schematic)
At the start: 34 parts, among them J1 Conn_01x02_Pin, J10 Conn_01x04_Pin, J11 Conn_01x04_Pin, J12 Conn_01x02_Pin, J13 Conn_01x04_Pin, J14 Conn_01x06_Pin, J15 Conn_01x04_Pin, J2 Conn_01x04_Pin, J3 Conn_01x02_Pin, J4 Conn_01x04_Pin, J5 Conn_01x02_Pin, J6 Conn_01x02_Pin, J7 Conn_01x02_Pin, J8 Conn_01x03_Pin, J9 Conn_01x03_Pin, U1 ESP32-S3-WROOM-1

Commit message: Staging
Parts:
- removed J8, J9: Conn_01x03_Pin, Connector_JST:JST_PH_B3B-PH-K_1x03_P2.00mm_Vertical, symbol Connector:Conn_01x03_Pin
- added D1: RED, Diode_SMD:D_0805_2012Metric_Pad1.15x1.40mm_HandSolder, symbol Device:LED
- added J8, J9: Conn_01x02_Pin, Connector_JST:JST_PH_B2B-PH-K_1x02_P2.00mm_Vertical, symbol Connector:Conn_01x02_Pin
- added R1: 150R, Resistor_SMD:R_0603_1608Metric_Pad0.98x0.95mm_HandSolder, symbol Device:R_Small
- added SW1: SW_Push, Easy:Button Aliexpress 4x4, symbol Switch:SW_Push
- C1: value 220u -> 220u 16V; LCSC C4747974 -> (none)
- renumbered D1 to D2, D2 to D3, R1 to R2, R2 to R3, R3 to R4, R4 to R5, R5 to R6, R6 to R7, R7 to R8, R8 to R9
Connections:
- net 3V3: now also J8.2 (Pin_2), J9.2 (Pin_2)
- net EN: now also SW1.1
- net GND: now also D1.1 (K), J8.1 (Pin_1), J9.1 (Pin_1), SW1.2
- net ACTIVE: now reaches U1.29 (SPIIO7/GPIO36/FSPICLK/SUBSPICLK)
- net ACTIVE: now also R1.1
- net PROCESS renamed FILTER
- new net: D1.2 (A), R1.2
Other:
- note removed: "PI6CV304"
- moved on the sheet: C3, C4, D2, D3, J1, J10, J11, J12, J13, J14, J15, J2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
