File: pcbs/plate-amp/1.1/plate-amp.kicad_pcb (KiCad board)
At the start: 2 copper layers, 75 x 95 mm, 95 parts, among them J1 Conn_01x02_Pin, J2 Conn_01x02_Pin, J3 Conn_01x02_Pin, J4 Conn_01x02_Pin, J5 Conn_01x02_Pin, J6 Conn_01x03_Pin, J7 Conn_01x04_Pin, J8 Conn_01x02_Pin, J9 Conn_01x02_Pin, U3 TPA3255DDV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

Commit message: Staging
Other:
- board text added: "PLATE 1.1"
- board text removed: "PLATE 1.0"
