File: pcbs/plate-amp/1.1/plate-amp.kicad_sch (KiCad schematic)
At the start: 95 parts, among them J1 Conn_01x02_Pin, J2 Conn_01x02_Pin, J3 Conn_01x02_Pin, J4 Conn_01x02_Pin, J5 Conn_01x02_Pin, J6 Conn_01x03_Pin, J7 Conn_01x04_Pin, J8 Conn_01x02_Pin, J9 Conn_01x02_Pin, U3 TPA3255DDV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

Commit message: Staging
Changed lines of the file:
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@@
 (kicad_sch
-	(version 20231120)
+	(version 20250114)
 	(generator "eeschema")
-	(generator_version "8.0")
+	(generator_version "9.0")
 	(paper "A2")
 	(junction
@@
 		)
 	)
+	(embedded_fonts no)
 )
