File: pcbs/psu-entry/1.1/psuentry.kicad_pcb (KiCad board)
At the start: 2 copper layers, 85 x 55 mm, 23 parts, among them J1 Conn_01x03_Pin, J2 Conn_01x02_Pin, J3 Conn_01x03_Pin, J4 Conn_01x03_Pin, J5 Conn_01x03_Pin, J6 Conn_01x06_Pin, U1 INA260, U2 INA260

Commit message: Updates
Connections:
- U1 pad 4: SDA -> PGND
- U1 pad 5: SDA -> 3V3
- U2 pad 4: SDA -> PGND
- U2 pad 5: SCL -> SDA
Routing:
- net PGND: track 376.6 -> 385.5 mm
- net SCL: track 60.4 -> 56.3 mm
- net SDA: track 55.8 -> 52.1 mm
- net 3V3: track 127.0 -> 129.9 mm
Other:
- board text added: "ENTRY 1.1"
- board text removed: "ENTRY 1.0"

Commit message: Staging
Parts:
- added J7: Conn_01x02_Pin, Connector_JST:JST_PH_B2B-PH-K_1x02_P2.00mm_Vertical, F.Cu at (96.1, 67.0)
- added J8: Conn_01x02_Pin, Connector_JST:JST_PH_B2B-PH-K_1x02_P2.00mm_Vertical, F.Cu at (103.2, 67.0)
- added J9: Conn_01x02_Pin, Connector_JST:JST_PH_B2B-PH-K_1x02_P2.00mm_Vertical, F.Cu at (110.4, 67.0)
- moved J1 70.2 mm to (165.6, 109.1), turned to 90 degrees
- moved C4 1.94 mm to (165.9, 93.3)
Routing:
- net PGND: track 385.5 -> 533.5 mm, vias 11 -> 14
- net DC_NEG: track 115.5 -> 47.0 mm
- net 3V3: track 129.9 -> 134.6 mm
- net SCL: track 56.3 -> 52.4 mm, vias 7 -> 6
- net DC_POS: track 58.7 -> 57.2 mm
- net DC_POS_POW: track 31.2 -> 32.3 mm
Other:
- board text added: "CHASSIS_GND"
- board text added: "SM_GND"
- board text added: "TO_MULTIPSU"
- board text removed: "GND"
- board text removed: "TO_DIGPSU"
