File: pcbs/spdif-cs8416/1.0/spdif-cs8416.kicad_sch (KiCad schematic)
At the start: 59 parts, among them J1 Conn_01x04_Pin, J10 Conn_01x05_Pin, J11 Conn_01x04_Pin, J12 Conn_01x02_Pin, J2 Conn_01x02_Pin, J3 Conn_01x02_Pin, J4 Conn_01x02_Pin, J5 Conn_01x02_Pin, J6 Conn_01x03_Pin, J7 Conn_01x02_Pin, J8 Conn_01x02_Pin, J9 Conn_01x02_Pin, U1 DA101C_C6931652, U2 ZLDO1117QG33TA, U3 DA101C_C6931652, U4 CS8416-xZZ, U5 DA101C_C6931652, X1 DFA-S3

Commit message: Staging
Parts:
- added J13: Conn_01x02_Pin, Connector_JST:JST_PH_B2B-PH-K_1x02_P2.00mm_Vertical, symbol Connector:Conn_01x02_Pin
- C10: renamed from C9; value 0.01u -> 0.1u; footprint Capacitor_SMD:C_0805_2012Metric -> Capacitor_SMD:C_0805_2012Metric_Pad1.18x1.45mm_HandSolder
- C14: Mouser (none) -> 80-C0805C223J3GECLR
- C16, C8: value 0.01u -> 0.1u; footprint Capacitor_SMD:C_0805_2012Metric -> Capacitor_SMD:C_0805_2012Metric_Pad1.18x1.45mm_HandSolder
- C4: footprint Capacitor_SMD:C_0805_2012Metric -> Capacitor_SMD:C_0805_2012Metric_Pad1.18x1.45mm_HandSolder
- R11: renamed from R12; footprint Resistor_SMD:R_0603_1608Metric_Pad0.98x0.95mm_HandSolder -> Resistor_SMD:R_0805_2012Metric_Pad1.20x1.40mm_HandSolder; Mouser (none) -> 603-RT0805FRE0775RL
- R12: renamed from R11; footprint Resistor_SMD:R_0603_1608Metric_Pad0.98x0.95mm_HandSolder -> Resistor_SMD:R_0805_2012Metric_Pad1.20x1.40mm_HandSolder; Mouser (none) -> 603-RT0805FRE133KL
- R5, R8: footprint Resistor_SMD:R_0603_1608Metric_Pad0.98x0.95mm_HandSolder -> Resistor_SMD:R_0805_2012Metric_Pad1.20x1.40mm_HandSolder; Mouser (none) -> 603-RT0805FRE0775RL
- R6: value 75R -> 300R
- R7: value 330R -> 550R
- TP1, TP2, TP3, TP4: footprint TestPoint:TestPoint_Plated_Hole_D2.0mm -> TestPoint:TestPoint_THTPad_D2.0mm_Drill1.0mm
- X1: value DFA-S3 -> 24.576 Mhz; footprint Oscillator:Oscillator_SMD_EuroQuartz_XO53-4Pin_5.0x3.2mm -> Oscillator:Oscillator_SMD_EuroQuartz_XO32-4Pin_3.2x2.5mm_HandSoldering; Mouser (none) -> 815-ASE24.576MHZLCT
- renumbered C10 to C9, J8 to J10, J9 to J11, J10 to J12, J11 to J2, J2 to J4, J4 to J5, J5 to J6, J6 to J7, J7 to J8, J12 to J9
Connections:
- net AGND: now also C5.1, J13.1 (Pin_1), J13.2 (Pin_2)
- net GND: no longer C5.1
Other:
- moved on the sheet: C1, C10, C11, C12, C13, C14, C15, C16, C17, C2, C3, C4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
