File: pcbs/spdif-cs8416/1.0/spdif-cs8416.kicad_pcb (KiCad board)
At the start: 2 copper layers, 85 x 55 mm, 59 parts, among them J1 Conn_01x04_Pin, J10 Conn_01x05_Pin, J11 Conn_01x04_Pin, J12 Conn_01x02_Pin, J2 Conn_01x02_Pin, J3 Conn_01x02_Pin, J4 Conn_01x02_Pin, J5 Conn_01x02_Pin, J6 Conn_01x03_Pin, J7 Conn_01x02_Pin, J8 Conn_01x02_Pin, J9 Conn_01x02_Pin, U1 DA101C_C6931652, U2 ZLDO1117QG33TA, U3 DA101C_C6931652, U4 CS8416-xZZ, U5 DA101C_C6931652, X1 DFA-S3

Commit message: Staging
Parts:
- added J13: Conn_01x02_Pin, Connector_JST:JST_PH_B2B-PH-K_1x02_P2.00mm_Vertical, F.Cu at (167.6, 109.9)
- C10: renamed from C9; value 0.01u -> 0.1u; footprint Capacitor_SMD:C_0805_2012Metric -> Capacitor_SMD:C_0805_2012Metric_Pad1.18x1.45mm_HandSolder
- C16, C8: value 0.01u -> 0.1u; footprint Capacitor_SMD:C_0805_2012Metric -> Capacitor_SMD:C_0805_2012Metric_Pad1.18x1.45mm_HandSolder
- C4: footprint Capacitor_SMD:C_0805_2012Metric -> Capacitor_SMD:C_0805_2012Metric_Pad1.18x1.45mm_HandSolder
- R11: renamed from R12; footprint Resistor_SMD:R_0603_1608Metric_Pad0.98x0.95mm_HandSolder -> Resistor_SMD:R_0805_2012Metric_Pad1.20x1.40mm_HandSolder
- R12: renamed from R11; footprint Resistor_SMD:R_0603_1608Metric_Pad0.98x0.95mm_HandSolder -> Resistor_SMD:R_0805_2012Metric_Pad1.20x1.40mm_HandSolder
- R5, R8: footprint Resistor_SMD:R_0603_1608Metric_Pad0.98x0.95mm_HandSolder -> Resistor_SMD:R_0805_2012Metric_Pad1.20x1.40mm_HandSolder
- R6: value 75R -> 300R
- R7: value 330R -> 550R
- TP1, TP2, TP3, TP4: footprint TestPoint:TestPoint_Plated_Hole_D2.0mm -> TestPoint:TestPoint_THTPad_D2.0mm_Drill1.0mm
- X1: value DFA-S3 -> 24.576 Mhz; footprint Oscillator:Oscillator_SMD_EuroQuartz_XO53-4Pin_5.0x3.2mm -> Oscillator:Oscillator_SMD_EuroQuartz_XO32-4Pin_3.2x2.5mm_HandSoldering
- moved J7 3.60 mm to (168.7, 98.1)
- moved R11 1.50 mm to (112.2, 101.4)
- moved R5 1.50 mm to (112.2, 75.6)
- moved R8 1.50 mm to (112.2, 88.9)
- moved C17 1.50 mm to (112.2, 106.7)
- moved C3 1.50 mm to (112.2, 81.1)
- moved C9 1.50 mm to (112.2, 93.8)
- moved J3 1.50 mm to (89.9, 77.0)
- moved J5 1.50 mm to (89.9, 89.9)
- moved J8 1.50 mm to (89.9, 102.8)
- moved U1 1.50 mm to (102.7, 78.4)
- moved U3 1.50 mm to (102.7, 91.2)
- moved U5 1.50 mm to (102.7, 104.1)
- moved C16 0.54 mm to (139.3, 103.5)
- moved C8 0.41 mm to (123.0, 92.8)
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- renumbered C10 to C9, J8 to J10, J9 to J11, J10 to J12, J11 to J2, J2 to J4, J4 to J5, J5 to J6, J6 to J7, J7 to J8, J12 to J9
Connections:
- C5 pad 1: GND -> AGND
Routing:
- net 3V3A: track 89.4 -> 78.9 mm
- net 5V: track 63.3 -> 59.9 mm
- net AGND: track 25.3 -> 27.6 mm, vias 8 -> 9
- net GND_IN: track 11.0 -> 12.5 mm
- net GPIO1: track 23.3 -> 24.1 mm
- net ADDR2: track 22.8 -> 22.0 mm
- net SPDIF2: track 16.2 -> 16.8 mm
- net SPDIF1: track 23.2 -> 23.8 mm
- net GPIO2: track 24.3 -> 23.9 mm, vias 4 -> 2
- net 3V3: track 142.5 -> 142.2 mm, vias 9 -> 7

Commit message: Updates
Other:
- board text added: "CS8416 1.1"
- board text removed: "CS8416 1.0"
