File: pcbs/psu-multi/1.3/multipsu.kicad_pcb (KiCad board)
At the start: 2 copper layers, 85 x 55 mm, 68 parts, among them J1 Conn_01x06_Pin, J2 Conn_01x03_Male, J3 Conn_01x02_Pin, J4 Conn_01x03_Pin, J5 Conn_01x03_Pin, J6 Conn_01x02_Pin, J7 Conn_01x03_Pin, U1 LM337_SOT223, U2 LM317_SOT-223, U3 ZLDO1117QG33TA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

Commit message: Updates
Parts:
- R1, R2: value 120R -> 240R
- R3, R4: value 1.2K -> 2.2K
- R5, R6: value 150R -> 330R
Connections:
- D1 pad 1: -16V -> PGND
- D1 pad 2: VN -> -16V
- R5 pad 1: PGND -> -16V
- R5 pad 2: -16V -> VN
Routing:
- net VN: track 58.4 -> 53.4 mm
