File: pcbs/psu-multi/1.4/multipsu.kicad_sch (KiCad schematic)
At the start: 68 parts, among them J1 Conn_01x06_Pin, J2 Conn_01x03_Male, J3 Conn_01x02_Pin, J4 Conn_01x03_Pin, J5 Conn_01x03_Pin, J6 Conn_01x02_Pin, J7 Conn_01x03_Pin, U1 LM337_SOT223, U2 LM317_SOT-223, U3 ZLDO1117QG33TA, U4 AMS1117-5.0, U5 NCP1117-12, U6 AP64351SP-13, U7 TMP100

Commit message: Updates
Parts:
- removed C10, C9: 1000u 16V, Capacitor_THT:CP_Radial_D8.0mm_P3.50mm, symbol Device:C_Polarized_Small
- removed C11, C21: 10U 50V, Capacitor_SMD:C_1206_3216Metric_Pad1.33x1.80mm_HandSolder, symbol Device:C_Polarized_Small
- removed C17, C18, C20: 10U, Capacitor_SMD:C_1206_3216Metric_Pad1.33x1.80mm_HandSolder, symbol Device:C_Polarized_Small
- removed C19: 10u, Capacitor_SMD:C_1206_3216Metric_Pad1.33x1.80mm_HandSolder, symbol Device:C_Small
- removed C22: 0.1u, Capacitor_SMD:C_0805_2012Metric_Pad1.18x1.45mm_HandSolder, symbol Device:C_Polarized_Small
- removed C7: 100u 50V, Capacitor_THT:CP_Radial_D8.0mm_P3.50mm, symbol Device:C_Polarized_Small
- removed D1, D2: 16V, Diode_SMD:D_SMA, symbol Device:D_Zener_Small
- removed R5, R6: 330R, Resistor_SMD:R_2512_6332Metric_Pad1.40x3.35mm_HandSolder, symbol Device:R_Small
- removed R7: 160K, Resistor_SMD:R_0603_1608Metric_Pad0.98x0.95mm_HandSolder, symbol Device:R_Small
- removed R8: 22K, Resistor_SMD:R_0603_1608Metric_Pad0.98x0.95mm_HandSolder, symbol Device:R_Small
- removed R9: 86.6k, Resistor_SMD:R_0603_1608Metric_Pad0.98x0.95mm_HandSolder, symbol Device:R_Small
- removed TP7, TP8, TP9: TestPoint, TestPoint:TestPoint_THTPad_D2.0mm_Drill1.0mm, symbol Connector:TestPoint
- removed U4: AMS1117-5.0, Package_TO_SOT_SMD:SOT-223-3_TabPin2, symbol Regulator_Linear:AMS1117-5.0
- removed U5: NCP1117-12, Package_TO_SOT_SMD:SOT-223, symbol Regulator_Linear:NCP1117-12_SOT223
- removed U6: AP64351SP-13, easyeda2kicad:SOIC-8_L4.9-W3.9-P1.27-LS6.0-BL-EP, symbol easyeda2kicad:AP64351SP-13
- added C18, C6, C7: 0.1u, Capacitor_SMD:C_0805_2012Metric_Pad1.18x1.45mm_HandSolder, symbol Device:C_Small
- added C24: 1000u 16V, Capacitor_THT:CP_Radial_D8.0mm_P3.50mm, symbol Device:C_Polarized_Small
- added C3: 22U 25V, Capacitor_SMD:C_1206_3216Metric_Pad1.33x1.80mm_HandSolder, symbol Device:C_Polarized_Small
- added C4, C5: 10U 50V, Capacitor_SMD:C_1206_3216Metric_Pad1.33x1.80mm_HandSolder, symbol Device:C_Polarized_Small
- added J3: Conn_01x02, Connector_PinHeader_2.54mm:PinHeader_1x02_P2.54mm_Vertical, symbol Connector_Generic:Conn_01x02
- added J4: Conn_01x02_Pin, Connector_JST:JST_PH_B2B-PH-K_1x02_P2.00mm_Vertical, symbol Connector:Conn_01x02_Pin
- added L2, L3: 6.8u, Inductor_SMD:L_Sunlord_MWSA0605S, symbol Device:L_Small
- added R1, R10, R3: 100K, Resistor_SMD:R_0603_1608Metric_Pad0.98x0.95mm_HandSolder, symbol Device:R_Small
- added R11, R4: 5.23K, Resistor_SMD:R_0603_1608Metric_Pad0.98x0.95mm_HandSolder, symbol Device:R_Small
- added R2: 13.7K, Resistor_SMD:R_0603_1608Metric_Pad0.98x0.95mm_HandSolder, symbol Device:R_Small
- added TP1: TestPoint, TestPoint:TestPoint_THTPad_D2.0mm_Drill1.0mm, symbol Connector:TestPoint
- added U1, U2, U7: LMR51430, Package_TO_SOT_SMD:SOT-23-6, symbol Regulator_Switching:LMR51430
- C1, C2: value 0.1U -> 22U 25V; footprint Capacitor_SMD:C_0805_2012Metric_Pad1.18x1.45mm_HandSolder -> Capacitor_SMD:C_1206_3216Metric_Pad1.33x1.80mm_HandSolder
- C12: value 10U 50V -> 22U 25V
- C13: value 0.22u -> 10U 50V; footprint Capacitor_SMD:C_0805_2012Metric_Pad1.18x1.45mm_HandSolder -> Capacitor_SMD:C_1206_3216Metric_Pad1.33x1.80mm_HandSolder
- C14: value 0.01u -> 22U 25V; footprint Capacitor_SMD:C_0805_2012Metric_Pad1.18x1.45mm_HandSolder -> Capacitor_SMD:C_1206_3216Metric_Pad1.33x1.80mm_HandSolder
- L1: value 10uH 21mOhm 5A -> 3.3u; footprint Inductor_SMD:L_Vishay_IHLP-4040 -> Inductor_SMD:L_Sunlord_MWSA0605S; Mouser 704-DR1040-7R0-R -> (none)
- R5: renamed from R10; value 1.7K -> 16K
- R6: renamed from R4; value 2.2K -> 1.6K; Mouser RC0603DR-072K2L -> RC0603FR-071K6L
- R7: renamed from R1; Mouser RT0603DRD07240RL -> RC0603FR-07240RL
- R8: renamed from R2; Mouser RT0603DRD07240RL -> RC0603FR-07240RL
- R9: renamed from R3; value 2.2K -> 1.6K; Mouser RC0603DR-072K2L -> RC0603FR-071K6L
- renumbered C5 to C10, C3 to C11, C6 to C16, C4 to C17, C23 to C19, C24 to C20, C25 to C21, C27 to C22, C26 to C23, C16 to C9, D3 to D1, J3 to J5, J4 to J6, J5 to J7, J6 to J8, J7 to J9, TP1 to TP2, TP4 to TP3, TP5 to TP4, TP3 to TP5, TP2 to TP7, U7 to U3, U3 to U4, U2 to U5, U1 to U6
Connections:
- net 12V: now also C16.1, J6.3 (Pin_3), TP7.1, U5.3 (VI), C4.1, C5.1, U1.3 (VIN), U1.5 (EN), U2.3 (VIN), U2.5 (EN)
- net 5V: now also C1.1, C15.1, L1.2, U4.3 (VI), R1.1
- net AGND: now also J3.1 (Pin_1); no longer C22.1, C23.2, J9.2 (Pin_2)
- net PGND: now also C1.2, C2.1, C24.2, C3.1, C4.2, C5.2, L2.2, R11.2, R2.2, R3.1, TP1.1, U1.1 (GND), U7.1 (GND); no longer C1.1, C2.2
- net VP: now also C13.1, D1.2 (A), U7.3 (VIN), U7.5 (EN); no longer C12.1
- net at L1.1: now also C6.2, U1.2 (SW)
- net 12V_OUT: now reaches C14.1
- net 12V_OUT: now also C12.1, J6.1 (Pin_1), C24.1, L3.2, R10.1
- net -16V renamed -12V
- net -12V: now also C2.2, C3.2, R4.2, U2.1 (GND); no longer C1.2
- removed net 16V: C16.1, C2.1, TP7.1, U5.3 (VI)
- removed net 7V_IN: C15.1, J6.3 (Pin_3), U4.3 (VI)
- removed net 7V_OUT: D1.2 (A), J6.1 (Pin_1), L1.2
- new net: R3.2, R4.1, U2.4 (FB)
- new net: C7.1, U2.6 (CB)
- new net: C7.2, L2.1, U2.2 (SW)
- new net: C18.2, L3.1, U7.2 (SW)
- new net: R10.2, R11.1, U7.4 (FB)
- new net: C18.1, U7.6 (CB)
- new net: R1.2, R2.1, U1.4 (FB)
- new net: C6.1, U1.6 (CB)
- new net AGND_INT: C22.1, C23.2, J3.2 (Pin_2), J4.1 (Pin_1), J4.2 (Pin_2), J9.2 (Pin_2)
Other:
- note added: "BUCK CONVERTERS"
- note added: "BULK CAPACITORS"
- moved on the sheet: C10, C11, C15, C17, C8, C9, J5, J6, J7, J8, J9, R5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
