File: pcbs/dac-pcm1690/1.0/dac.kicad_pcb (KiCad board)
At the start: 2 copper layers, 85 x 55 mm, 57 parts, among them J1 Conn_01x03_Pin, J10 Conn_01x02_Pin, J11 Conn_01x02_Pin, J12 Conn_01x04_Pin, J13 Conn_01x03_Pin, J14 Conn_01x04_Pin, J15 Conn_01x03_Pin, J16 Conn_01x03_Pin, J17 Conn_01x04_Pin, J18 Conn_01x02_Pin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

Commit message: UPdates
Parts:
- removed C10, C13, C15, C8: 0.1U, Capacitor_SMD:C_0805_2012Metric_Pad1.18x1.45mm_HandSolder
- removed C14, C16, C9: 10U, Capacitor_SMD:C_1206_3216Metric_Pad1.33x1.80mm_HandSolder
- removed C6, C7: 2.2u 25V, Capacitor_SMD:C_1206_3216Metric_Pad1.33x1.80mm_HandSolder
- removed J6, J8, J9: Conn_01x02_Pin, Connector_PinHeader_2.54mm:PinHeader_1x02_P2.54mm_Vertical
- removed R6, R7, R8: 4.7K, Resistor_SMD:R_0603_1608Metric_Pad0.98x0.95mm_HandSolder
- removed TP1, TP2, TP3: TestPoint, TestPoint:TestPoint_THTPad_D2.0mm_Drill1.0mm
- removed U4: PCM5122PW, Package_SO:TSSOP-28_4.4x9.7mm_P0.65mm
- added U5: PCM1690DCAR, easyeda2kicad:HTSSOP-48_L12.5-W6.1-P0.50-LS8.1-BL-EP-1, F.Cu at (81.5, 90.3)
Routing:
- net 3V3: track 140.3 -> 0.00 mm, vias 7 -> 0
- net 3V3A: track 91.8 -> 0.00 mm, vias 6 -> 0
- net LEFT_TWEETER: track 67.4 -> 0.00 mm, vias 2 -> 0
- net 5V: track 62.5 -> 0.00 mm, vias 2 -> 0
- net SDA: track 58.5 -> 0.00 mm, vias 2 -> 0
- net SCL: track 57.3 -> 0.00 mm, vias 2 -> 0
- net LEFT_WOOFER: track 50.1 -> 0.00 mm, vias 1 -> 0
- net SCLK: track 37.3 -> 0.00 mm
- net DATA: track 37.0 -> 0.00 mm, vias 1 -> 0
- net BCLK: track 37.0 -> 0.00 mm
- net LRCLK: track 36.7 -> 0.00 mm, vias 2 -> 0
- net XSMT_IN: track 33.3 -> 0.00 mm, vias 1 -> 0
- net XSMT: track 28.9 -> 0.00 mm, vias 3 -> 0
- net AGND: track 23.7 -> 0.00 mm, vias 10 -> 0
- net ADDR1: track 21.1 -> 0.00 mm
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Other:
- board text removed: "ADDR1"
- board text removed: "GND"
- board text removed: "XSMT"
