File: pcbs/dac-pcm1690/1.0/dac.kicad_sch (KiCad schematic)
At the start: 57 parts, among them J1 Conn_01x03_Pin, J10 Conn_01x02_Pin, J11 Conn_01x02_Pin, J12 Conn_01x04_Pin, J13 Conn_01x03_Pin, J14 Conn_01x04_Pin, J15 Conn_01x03_Pin, J16 Conn_01x03_Pin, J17 Conn_01x04_Pin, J18 Conn_01x02_Pin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

Commit message: UPdates
Parts:
- removed C15: 0.1U, Capacitor_SMD:C_0805_2012Metric_Pad1.18x1.45mm_HandSolder, symbol Device:C_Small
- removed C16: 10U, Capacitor_SMD:C_1206_3216Metric_Pad1.33x1.80mm_HandSolder, symbol Device:C_Small
- removed C6, C7: 2.2u 25V, Capacitor_SMD:C_1206_3216Metric_Pad1.33x1.80mm_HandSolder, symbol Device:C_Small
- removed J6, J8, J9: Conn_01x02_Pin, Connector_PinHeader_2.54mm:PinHeader_1x02_P2.54mm_Vertical, symbol Connector:Conn_01x02_Pin
- removed R8: 4.7K, Resistor_SMD:R_0603_1608Metric_Pad0.98x0.95mm_HandSolder, symbol Device:R_Small
- removed U4: PCM5122PW, Package_SO:TSSOP-28_4.4x9.7mm_P0.65mm, symbol Audio:PCM5122PW
- added U4: ~, symbol Custom:PCM1681
- added U5: PCM1690DCAR, easyeda2kicad:HTSSOP-48_L12.5-W6.1-P0.50-LS8.1-BL-EP-1, symbol easyeda2kicad:PCM1690DCAR
Connections:
- net ADDR2 is gone; now on net GND: R6.2
- net 3V3: now also U5.12 (VDD)
- net 5V: now also U5.25 (VCC1), U5.47 (VCC2)
- net AGND: now also U5.1 (RSV2), U5.27 (AGND1), U5.28 (RSV2), U5.3 (RSV2), U5.46 (AGND2), U5.5 (RSV2)
- net BCLK: now also U5.7 (BCK)
- net DATA: now also U5.8 (DIN1)
- net GND: now also U5.13 (DGND), U5.24 (MODE); no longer R6.1
- net LRCLK: now also U5.6 (LRCK)
- net SCL: now also U5.21 (MC/SCL/FMT)
- net SCLK: now also U5.14 (SCKI)
- net SDA: now also U5.20 (MD/SDA/DEMP)
- net XSMT: no longer names the net of R7.2
- net XSMT: now also U5.18 (AMUTEI)
- net XSMT_IN renamed RESET
- net RESET: now also R6.1, U5.15 (RST)
Other:
- note added: "DAC"
