File: pcbs/dac-pcm1792a/1.0/dac.kicad_pcb (KiCad board)
At the start: 2 copper layers, 85 x 55 mm, 74 parts, among them J1 Conn_01x03_Pin, J10 Conn_01x04_Pin, J11 Conn_01x03_Pin, J12 Conn_01x04_Pin, J13 Conn_01x03_Pin, J14 Conn_01x04_Pin, J2 Conn_01x03_Pin, J3 Conn_01x03_Pin, J4 Conn_01x02_Pin, J5 Conn_01x03_Pin, J6 Conn_01x03_Pin, J7 Conn_01x02_Pin, J8 Conn_01x02_Pin, J9 Conn_01x02_Pin, U1 OPA1656, U2 OPA1656, U3 OPA1656, U4 PCM1792A, Y1 ASE-xxxMHz

Commit message: Updates
Parts:
- added C11: 10u, Capacitor_SMD:C_1206_3216Metric_Pad1.33x1.80mm_HandSolder, F.Cu at (109.6, 79.9)
- added C5: 10u, Capacitor_SMD:C_1206_3216Metric_Pad1.33x1.80mm_HandSolder, F.Cu at (88.5, 73.8)
- R17: value 500R -> 1.5K
- R8: value 330R -> 10K
- moved C6 0.95 mm to (92.0, 74.4)
- moved R4 0.06 mm to (102.2, 70.4)
- moved R5 0.06 mm to (121.6, 70.4)
- renumbered C9 to C10, C10 to C12, C11 to C13, C12 to C14, C13 to C15, C14 to C16, C15 to C17, C16 to C18, C17 to C19, C18 to C20, C19 to C21, C20 to C22, C21 to C23, C22 to C24, C23 to C25, C24 to C26, C26 to C27, C25 to C28, C27 to C29, C28 to C30, C5 to C6, C6 to C7, C7 to C8, C8 to C9
Routing:
- net Net-(C18-Pad1): track 31.3 -> 20.8 mm
- net SCL: track 36.9 -> 44.1 mm, vias 2 -> 1
- net GND: track 10.8 -> 17.7 mm, vias 5 -> 14
- net VNEG: track 109.9 -> 103.9 mm, vias 8 -> 2
- net AGND: track 39.5 -> 44.6 mm, vias 28 -> 24
- net MCLK: track 19.4 -> 24.2 mm, vias 3 -> 4
- net 5V: track 116.3 -> 111.7 mm, vias 2 -> 0
- net VPOS: track 103.2 -> 107.4 mm, vias 7 -> 1
- net Net-(C4-Pad2): track 31.3 -> 27.2 mm, vias 0 -> 1
- net Net-(C2-Pad1): track 21.5 -> 17.7 mm, vias 0 -> 1
- net IOUTR-: track 39.0 -> 42.0 mm, vias 1 -> 3
- net Net-(C3-Pad2): track 57.3 -> 60.1 mm, vias 4 -> 3
- net SDA: track 41.3 -> 43.6 mm, vias 2 -> 1
- net IOUTL+: track 23.9 -> 26.1 mm, vias 2 -> 1
- net GND_IN: track 24.8 -> 26.3 mm, vias 1 -> 2
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- added copper zone on In2.Cu, net AGND
- added copper zone on In1.Cu, net GND
Other:
- copper layers 2 -> 4
