File: pcbs/psu-monitor/1.2/monitor.kicad_pcb (KiCad board)
At the start: 2 copper layers, 85 x 55 mm, 23 parts, among them J1 Conn_01x03_Pin, J2 Conn_01x03_Pin, J3 Conn_01x02_Pin, J4 Conn_01x03_Pin, J5 Conn_01x02_Pin, J6 Conn_01x02_Pin, J7 Conn_01x02_Pin, J8 Conn_01x03_Pin, J9 Conn_01x03_Pin, U1 INA260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

Commit message: Updates
Connections:
- U4 pad 8: unconnected-(U4-SDA-Pad8) -> SDA
Routing:
- net SDA: track 76.5 -> 78.2 mm
Other:
- board text added: "MONITOR 1.2"
- board text removed: "MONITOR 1.1"
