File: pcbs/psu-monitor/1.2/monitor.kicad_sch (KiCad schematic)
At the start: 23 parts, among them J1 Conn_01x03_Pin, J2 Conn_01x03_Pin, J3 Conn_01x02_Pin, J4 Conn_01x03_Pin, J5 Conn_01x02_Pin, J6 Conn_01x02_Pin, J7 Conn_01x02_Pin, J8 Conn_01x03_Pin, J9 Conn_01x03_Pin, U1 INA260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

Commit message: Updates
Connections:
- net SDA: now also U4.8 (SDA)
Changed lines of the file:
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@@
+		)
+	)
+	(global_label "SDA"
+		(shape input)
+		(at 407.67 67.31 0)
+		(fields_autoplaced yes)
+		(effects
+			(font
+				(size 1.27 1.27)
+			)
+			(justify left)
+		)
+		(property "Intersheetrefs" "${INTERSHEET_REFS}"
+			(at 414.2233 67.31 0)
+			(effects
+				(font
+					(size 1.27 1.27)
+				)
+				(justify left)
+				(hide yes)
+			)
 		)
 	)
