File: pcbs/psu/digital/digital.kicad_pcb (KiCad board)
At the start: 2 copper layers, 85 x 55 mm, 33 parts, among them J1 Conn_01x03, J2 Conn_01x03, J3 Conn_01x03, U1 TMP100, U2 AZ1117-3.3, U3 AZ1117-5.0, U4 AZ1117-5.0

Commit message: Updates
Parts:
- removed C5: 4700u, Capacitor_THT:CP_Radial_D16.0mm_P7.50mm
- added C12: 10u, Capacitor_SMD:C_1206_3216Metric_Pad1.33x1.80mm_HandSolder, F.Cu at (138.5, 57.5)
- moved R1 29.4 mm to (115.5, 58.9), turned to 90 degrees
- moved D1 25.0 mm to (115.5, 55.0), turned to -90 degrees
- moved TP1 24.2 mm to (115.5, 63.5), turned to 90 degrees
- moved J2 21.8 mm to (96.8, 54.5)
- moved C1 16.0 mm to (97.5, 78.2), turned to 90 degrees
- moved C2 16.0 mm to (115.7, 78.1), turned to 90 degrees
- moved C8 16.0 mm to (97.5, 95.1), turned to 90 degrees
- moved C9 16.0 mm to (115.7, 95.0), turned to 90 degrees
- moved R2 14.3 mm to (111.0, 59.0), turned to 90 degrees
- moved J1 13.0 mm to (122.0, 52.5)
- moved H1 10.0 mm to (90.5, 52.5)
- moved H3 10.0 mm to (90.5, 102.5)
- moved TP2 9.75 mm to (111.0, 63.5), turned to 90 degrees
- moved D2 9.33 mm to (111.0, 55.0), turned to -90 degrees
Routing:
- net 5V: track 144.0 -> 110.3 mm, vias 3 -> 2
- net 7V: track 135.8 -> 110.8 mm
- net 3V3: track 99.8 -> 120.8 mm, vias 2 -> 4
- net 3V3_OUT: track 38.0 -> 25.1 mm, vias 3 -> 2
- net SDA: track 31.0 -> 18.5 mm, vias 1 -> 2
- net SCL: track 34.3 -> 22.0 mm, vias 1 -> 2
- net GND: track 41.4 -> 41.3 mm, vias 88 -> 87
Other:
- board size 85 x 55 mm -> 75 x 55 mm
