File: pcbs/psu/fanout/monitors.kicad_sch (KiCad schematic)
At the start: 18 parts, among them J10 Conn_01x03, J11 Conn_01x03, J13 Conn_01x03, J15 Conn_01x03, J16 Conn_01x02, J17 Conn_01x02, J6 Conn_01x03, J7 Conn_01x03, J8 Conn_01x03, J9 Conn_01x03, U1 INA260, U2 INA260, U3 INA260, U4 INA260

Commit message: Updates
Parts:
- removed J10, J11: Conn_01x03, Connector_JST:JST_VH_B3P-VH-B_1x03_P3.96mm_Vertical, symbol Connector_Generic:Conn_01x03
- removed J13: Conn_01x03, Connector_JST:JST_PH_B3B-PH-K_1x03_P2.00mm_Vertical, symbol Connector_Generic:Conn_01x03
- removed J17: Conn_01x02, Connector_JST:JST_PH_B2B-PH-K_1x02_P2.00mm_Vertical, symbol Connector_Generic:Conn_01x02
- removed U1, U2, U3, U4: INA260, Package_SO:TSSOP-16_4.4x5mm_P0.65mm, symbol Sensor:INA260
- added J1, J2, J3, J4, J5, J6, J7, J8: Conn_01x03, TerminalBlock_Phoenix:TerminalBlock_Phoenix_PT-1,5-3-3.5-H_1x03_P3.50mm_Horizontal, symbol Connector_Generic:Conn_01x03
- added J10: Conn_01x02, Connector_JST:JST_VH_B2P-VH-B_1x02_P3.96mm_Vertical, symbol Connector_Generic:Conn_01x02
- added J11, J12, J18: Conn_01x02, Connector_JST:JST_PH_B2B-PH-K_1x02_P2.00mm_Vertical, symbol Connector_Generic:Conn_01x02
- added J17: Conn_01x04, Connector_JST:JST_PH_B4B-PH-K_1x04_P2.00mm_Vertical, symbol Connector_Generic:Conn_01x04
- added R1, R2: 4.7k, Resistor_SMD:R_0805_2012Metric_Pad1.20x1.40mm_HandSolder, symbol Device:R_Small
- added TP1, TP2, TP3, TP4: TestPoint, TestPoint:TestPoint_THTPad_2.5x2.5mm_Drill1.2mm, symbol Connector:TestPoint
- J15: footprint Connector_JST:JST_PH_B3B-PH-K_1x03_P2.00mm_Vertical -> Connector_JST:JST_VH_B3P-VH-B_1x03_P3.96mm_Vertical
- J9: footprint Connector_JST:JST_VH_B3P-VH-B_1x03_P3.96mm_Vertical -> TerminalBlock_Phoenix:TerminalBlock_Phoenix_PT-1,5-3-3.5-H_1x03_P3.50mm_Horizontal
- renumbered J6 to J13, J7 to J14, J8 to J16, J16 to J19
Connections:
- net OPAMP+OUT is gone; now on net V+: J9.3 (Pin_3)
- net 3V3: now also J4.1 (Pin_1), J5.1 (Pin_1), J6.1 (Pin_1)
- net 5V: now also J4.3 (Pin_3), J5.3 (Pin_3), J6.3 (Pin_3)
- net GND: now also J15.2 (Pin_2), J1.2 (Pin_2), J10.1 (Pin_1), J10.2 (Pin_2), J2.2 (Pin_2), J3.2 (Pin_2), J4.2 (Pin_2), J5.2 (Pin_2), J6.2 (Pin_2), J7.2 (Pin_2), J8.2 (Pin_2), R1.2, R2.2, TP1.1, TP2.1, TP3.1, TP4.1
- net OPAMP+: now also J1.3 (Pin_3), J2.3 (Pin_3), J3.3 (Pin_3)
- net OPAMP-: now also J1.1 (Pin_1), J2.1 (Pin_1), J3.1 (Pin_1); no longer J9.1 (Pin_1)
- net SCL: now also J12.1 (Pin_1), J18.1 (Pin_1); no longer J15.2 (Pin_2)
- net SDA: now also J12.2 (Pin_2), J18.2 (Pin_2); no longer J15.3 (Pin_3)
- net V+: now also J7.3 (Pin_3)
- net V-: now also J9.1 (Pin_1), J7.1 (Pin_1)
- net 3V3_OUT renamed 3V3_STANDBY
- net 3V3_STANDBY: now also J8.1 (Pin_1)
- new net 5V_STANDBY: J15.3 (Pin_3), J8.3 (Pin_3)
- new net EXT1: J11.1 (Pin_1), J17.1 (Pin_1), R1.1
- new net EXT2: J11.2 (Pin_2), J17.2 (Pin_2), R2.1
- new net EXT3: J17.3 (Pin_3)
- new net EXT4: J17.4 (Pin_4)
