File: pcbs/psu/monitor/monitors.kicad_pcb (KiCad board)
At the start: 2 copper layers, 95 x 75 mm, 39 parts, among them J1 Conn_01x02, J10 Conn_01x03, J11 Conn_01x03, J12 Conn_01x03, J13 Conn_01x03, J14 Conn_01x04, J15 Conn_01x03, J16 Conn_01x02, J17 Conn_01x02, J18 Conn_01x02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

Commit message: Updates
Parts:
- removed D1, D2, D3: 1N4001, Diode_SMD:D_SMA
- removed J1: Conn_01x02, Connector_JST:JST_VH_B2P-VH-B_1x02_P3.96mm_Vertical
- removed J12, J2, J3, J4, J5: Conn_01x03, TerminalBlock_Phoenix:TerminalBlock_Phoenix_PT-1,5-3-3.5-H_1x03_P3.50mm_Horizontal
- removed J14: Conn_01x04, Connector_JST:JST_PH_B4B-PH-K_1x04_P2.00mm_Vertical
- removed J18: Conn_01x02, Connector_JST:JST_PH_B2B-PH-K_1x02_P2.00mm_Vertical
- removed J19: Conn_01x03, Connector_JST:JST_PH_B3B-PH-K_1x03_P2.00mm_Vertical
- removed K1, K2, K3: G2RL-2, Relay_THT:Relay_DPDT_Omron_G2RL-2
- removed Q1, Q2, Q3: BC847, Package_TO_SOT_SMD:SOT-23
- removed R1, R2, R3: 1k, Resistor_SMD:R_0805_2012Metric_Pad1.20x1.40mm_HandSolder
- J10, J11, J9: footprint TerminalBlock_Phoenix:TerminalBlock_Phoenix_PT-1,5-3-3.5-H_1x03_P3.50mm_Horizontal -> Connector_JST:JST_VH_B3P-VH-B_1x03_P3.96mm_Vertical
- moved J11 82.3 mm to (93.3, 83.0), turned to 0 degrees
- moved J9 41.4 mm to (128.7, 83.0), turned to 0 degrees
- moved J10 40.5 mm to (164.1, 83.0), turned to 0 degrees
- moved J17 37.0 mm to (118.3, 81.0), turned to 0 degrees
- moved H1 30.0 mm to (87.5, 81.0)
- moved H2 30.0 mm to (177.5, 81.0)
- moved J15 26.9 mm to (176.6, 97.0), turned to 90 degrees
- moved U2 14.3 mm to (124.4, 95.6)
- moved U4 14.0 mm to (135.1, 95.6)
- moved U3 13.7 mm to (145.8, 95.6)
- moved U1 10.1 mm to (113.7, 95.6)
- moved J16 6.90 mm to (118.3, 110.0)
- moved J7 3.93 mm to (128.7, 108.0)
- moved J13 2.40 mm to (109.2, 110.0)
- moved J8 0.92 mm to (164.1, 108.0)
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Connections:
- J10 pad 1: 3V3_OUT_SW -> 3V3_OUT
- J10 pad 3: 5V_OUT_SW -> 5V_OUT
- J11 pad 1: 3V3_OUT_SW -> V-
- J11 pad 3: 5V_OUT_SW -> V+OUT
- J9 pad 1: OPAMP-_SW -> OPAMP-
- J9 pad 3: OPAMP+OUT_SW -> OPAMP+OUT
Routing:
- net GND: track 402.4 -> 180.7 mm, vias 25 -> 18
- net SCL: track 155.3 -> 98.0 mm, vias 13 -> 3
- net 5V_OUT_SW: track 55.1 -> 0.00 mm, vias 1 -> 0
- net DIGITAL_ON: track 54.3 -> 0.00 mm, vias 2 -> 0
- net OPAMP+OUT_SW: track 53.1 -> 0.00 mm, vias 1 -> 0
- net OPAMP_ON: track 49.2 -> 0.00 mm, vias 2 -> 0
- net 3V3_OUT_SW: track 48.7 -> 0.00 mm
- net SDA: track 149.3 -> 101.4 mm, vias 13 -> 3
- net OPAMP-_SW: track 47.2 -> 0.00 mm
- net 5V_OUT: track 143.5 -> 99.5 mm
- net Net-(D2-A): track 42.4 -> 0.00 mm, vias 3 -> 0
- net V+OUT_SW: track 37.8 -> 0.00 mm, vias 1 -> 0
- net 3V3_OUT: track 194.9 -> 157.4 mm, vias 15 -> 22
- net V-: track 62.4 -> 25.0 mm, vias 1 -> 0
- net Net-(D3-A): track 37.0 -> 0.00 mm, vias 2 -> 0
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- removed copper zone on B.Cu, net GND
Other:
- board size 95 x 75 mm -> 95 x 35 mm
- board text added: "AMP_POWER_IN"
- board text added: "AMP_POWER_OUT"
- board text added: "DIGITAL_POWER_IN"
- board text added: "DIGITAL_POWER_OUT"
- board text added: "OPAMP_POWER_IN"
- board text added: "OPAMP_POWER_OUT"
- board text removed: "AMP POWER"
- board text removed: "CHASSIS"
- board text removed: "DIGITAL POWER"
- board text removed: "DIGITAL_POWER"
- board text removed: "MONOBLOCK_POWER"
- board text removed: "OPAMP POWER"
- board text removed: "OPAMP_POWER"
- board text removed: "TO RECTIFIER"
- board text removed: "uPROC_SIG"
