File: pcbs/psu/relays/monitors.kicad_sch (KiCad schematic)
At the start: 38 parts, among them J1 Conn_01x04, J10 Conn_01x03, J11 Conn_01x03, J12 Conn_01x03, J18 Conn_01x02, J19 Conn_01x02, J6 Conn_01x03, J7 Conn_01x03, J8 Conn_01x03, J9 Conn_01x03, K1 G2RL-2, K2 G2RL-2, K3 G2RL-2, Q1 BC847, Q2 BC847, Q3 BC847, U1 MCP23008-xSS

Commit message: All changes
Parts:
- added J10: Conn_01x02, Connector_JST:JST_PH_B2B-PH-K_1x02_P2.00mm_Vertical, symbol Connector_Generic:Conn_01x02
- added J12: Conn_01x02, symbol Connector_Generic:Conn_01x02
- added R10: 4.7k, Resistor_SMD:R_0805_2012Metric_Pad1.20x1.40mm_HandSolder, symbol Device:R_Small
- renumbered D4 to D1, D5 to D2, D6 to D3, D1 to D4, D2 to D5, D3 to D6, J19 to J11, J18 to J2, J9 to J3, J10 to J4, J12 to J5, J11 to J6, J6 to J7, J7 to J8, J8 to J9, Q3 to Q2, Q2 to Q3, R7 to R1, R8 to R2, R9 to R3, R1 to R4, R2 to R5, R3 to R6, R4 to R7, R6 to R8, R5 to R9
Connections:
- net 3V3: now also R10.1
- net DGND: now also J10.1 (Pin_1)
- net RESET: now reaches U1.6 (~{RESET})
- net RESET: now also J10.2 (Pin_2), R10.2
