File: pcbs/psu/uproc/uproc.kicad_sch (KiCad schematic)
At the start: 36 parts, among them J1 Conn_01x03, J19 Conn_01x03, J2 Conn_01x04, J3 Conn_01x04, J4 Conn_01x02, J5 Conn_01x02, J6 Conn_01x06, J7 Conn_01x02, SW1 SW_Push, SW2 SW_Push, U1 ESP32-S3-WROOM-1, U2 TCA9517D

Commit message: Updates
Parts:
- added C1, C2: 10u, Capacitor_SMD:C_1206_3216Metric_Pad1.33x1.80mm_HandSolder, symbol Device:C_Small
- added C3, C5: 0.1u, Capacitor_SMD:C_0805_2012Metric_Pad1.18x1.45mm_HandSolder, symbol Device:C_Small
- added D3: BLUE, LED_SMD:LED_0805_2012Metric_Pad1.15x1.40mm_HandSolder, symbol Device:LED_Small
- added J7: Conn_01x04, Connector_JST:JST_PH_B4B-PH-K_1x04_P2.00mm_Vertical, symbol Connector_Generic:Conn_01x04
- added R16: 330R, Resistor_SMD:R_0805_2012Metric_Pad1.20x1.40mm_HandSolder, symbol Device:R_Small
- renumbered C2 to C4, C1 to C6, C3 to C7, J5 to J1, J7 to J2, J1 to J3, J19 to J4, J4 to J5, J3 to J8, J2 to J9, R10 to R1, R12 to R10, R7 to R11, R9 to R12, R8 to R13, R2 to R14, R5 to R15, R4 to R2, R6 to R3, R3 to R4, R1 to R5, R11 to R6, R15 to R7, R14 to R8, R13 to R9
Connections:
- net 3V3: now also C1.2, C5.1, J7.2 (Pin_2)
- net 5V: now also C2.2, C3.2
- net GND: now also C1.1, C2.1, C3.1, C5.2, D3.1 (K), J7.1 (Pin_1)
- net SCL: now also J7.3 (Pin_3)
- net SDA: now also J7.4 (Pin_4)
- net LED: now reaches U1.20 (GPIO12/TOUCH12/ADC2_CH1/FSPICLK/FSPIIO6/SUBSPICLK)
- net LED: now also R16.1
- new net: D3.2 (A), R16.2

Commit message: All changes
Parts:
- removed J2: Conn_01x02, Connector_JST:JST_PH_B2B-PH-K_1x02_P2.00mm_Vertical, symbol Connector_Generic:Conn_01x02
- removed J4: Conn_01x03, Connector_JST:JST_PH_B3B-PH-K_1x03_P2.00mm_Vertical, symbol Connector_Generic:Conn_01x03
- removed R10, R7, R8, R9: 4.7k, Resistor_SMD:R_0805_2012Metric_Pad1.20x1.40mm_HandSolder, symbol Device:R_Small
- added C1: 0.1u, Capacitor_SMD:C_0805_2012Metric_Pad1.18x1.45mm_HandSolder, symbol Device:C_Small
- added J10, J12, J15, J16, J7: Conn_01x02, Connector_JST:JST_PH_B2B-PH-K_1x02_P2.00mm_Vertical, symbol Connector_Generic:Conn_01x02
- added J11, J3, J4: Conn_01x04, Connector_JST:JST_PH_B4B-PH-K_1x04_P2.00mm_Vertical, symbol Connector_Generic:Conn_01x04
- added J17, J18: Conn_01x02, Connector_PinHeader_2.54mm:PinHeader_1x02_P2.54mm_Vertical, symbol Connector_Generic:Conn_01x02
- added J2: Conn_01x03, Connector_JST:JST_PH_B3B-PH-K_1x03_P2.00mm_Vertical, symbol Connector_Generic:Conn_01x03
- added U1: TMP100, Package_TO_SOT_SMD:SOT-23-6, symbol Sensor_Temperature:TMP100
- renumbered C1 to C3, C3 to C4, C6 to C5, C4 to C6, C5 to C8, D3 to D1, D1 to D2, D2 to D3, J8 to J13, J9 to J14, J3 to J5, J5 to J6, J6 to J8, J7 to J9, R4 to R1, R15 to R10, R5 to R11, R6 to R12, R1 to R3, R3 to R4, R16 to R5, R11 to R6, R12 to R7, R13 to R8, R14 to R9, U1 to U2, U2 to U3
Connections:
- net 3V3: now also C1.2, J10.2 (Pin_2), J12.1 (Pin_1), J18.2 (Pin_2), J2.1 (Pin_1), U1.3 (ADD1), U1.4 (V+), U1.5 (ADD0)
- net 5V: now also J2.3 (Pin_3)
- net GND: now also C1.1, J10.1 (Pin_1), J15.1 (Pin_1), J16.1 (Pin_1), J18.1 (Pin_1), J2.2 (Pin_2), U1.2 (GND)
- net SCL: now also J4.3 (Pin_3), U1.1 (SCL)
- net SDA: now also J4.4 (Pin_4), U1.6 (SDA)
- net SDCARD_CD: now reaches U2.10 (GPIO17/U1TXD/ADC2_CH6)
- net GPIO_RESET: now reaches U2.11 (GPIO18/U1RXD/ADC2_CH7/CLK_OUT3)
- net GPIO_RESET: now also J7.2 (Pin_2)
- net DN: now reaches U2.13 (GPIO19/U1RTS/ADC2_CH8/CLK_OUT2/USB_D-)
- net DN: now also J4.2 (Pin_2)
- net DP: now reaches U2.14 (GPIO20/U1CTS/ADC2_CH9/CLK_OUT1/USB_D+)
- net DP: now also J4.1 (Pin_1)
- net FROM_TOGGLE: now reaches U2.22 (GPIO14/TOUCH14/ADC2_CH3/FSPIWP/FSPIDQS/SUBSPIWP)
- net FROM_TOGGLE: now also J12.2 (Pin_2)
- net EXT1: now reaches U2.24 (GPIO47/SPICLK_P/SUBSPICLK_P_DIFF)
- net EXT1: now also J15.2 (Pin_2), J17.1 (Pin_1)
- net EXT2: now reaches U2.25 (GPIO48/SPICLK_N/SUBSPICLK_N_DIFF)
- net EXT2: now also J16.2 (Pin_2), J17.2 (Pin_2)
- net DIGITAL_ON renamed SPI_MOSI
- net SPI_MOSI: now also J11.1 (Pin_1), J3.3 (Pin_3)
- net FUTURE renamed SPI_CS2
- net SPI_CS2: now also J3.1 (Pin_1)
- net MONOBLOCK_ON renamed SPI_CLK
- net SPI_CLK: now also J11.3 (Pin_3), J3.2 (Pin_2)
- net OPAMP_ON renamed SPI_MISO
- net SPI_MISO: now also J11.2 (Pin_2), J3.4 (Pin_4)
- net POWER_ON renamed SPI_CS1
- net SPI_CS1: now also J11.4 (Pin_4)
Other:
- moved on the sheet: J13, J14, R10
