File: pcbs/_final_proto/dac-pcm1681/1.0/dac.kicad_pcb (KiCad board)
At the start: 2 copper layers, 75 x 55 mm, 67 parts, among them J1 Conn_01x03_Pin, J10 Conn_01x02_Pin, J11 Conn_01x03_Pin, J12 Conn_01x03_Pin, J13 Conn_01x02_Pin, J14 Conn_01x02_Pin, J15 Conn_01x02_Pin, J16 Conn_01x03_Pin, J17 Conn_01x02_Pin, J18 Conn_01x04_Pin, J19 Conn_01x04_Pin, J2 Conn_01x02_Pin, J20 Conn_01x02_Pin, J21 Conn_01x03_Pin, J22 Conn_01x04_Pin, J23 Conn_01x02_Pin, J3 Conn_01x02_Pin, J4 Conn_01x03, J5 Conn_01x03_Pin, J6 Conn_01x02_Pin, J7 Conn_01x02_Pin, J8 Conn_01x02_Pin, J9 Conn_01x02_Pin, U1 TPS7A0533PDBV, U2 PCM5122PW

Commit message: Working code
Parts:
- removed C11, C13, C17: 0.1U, Capacitor_SMD:C_0805_2012Metric_Pad1.18x1.45mm_HandSolder
- removed C14, C18: 10U, Capacitor_SMD:C_1206_3216Metric_Pad1.33x1.80mm_HandSolder
- removed C6, C7: 22U-47U, Capacitor_SMD:C_1206_3216Metric_Pad1.33x1.80mm_HandSolder
- removed J1, J21: Conn_01x03_Pin, Connector_JST:JST_PH_B3B-PH-K_1x03_P2.00mm_Vertical
- removed J17, J2, J3: Conn_01x02_Pin, Connector_JST:JST_PH_B2B-PH-K_1x02_P2.00mm_Vertical
- removed J22: Conn_01x04_Pin, Connector_PinHeader_2.54mm:PinHeader_1x04_P2.54mm_Vertical
- removed J23, J6, J9: Conn_01x02_Pin, Connector_PinHeader_2.54mm:PinHeader_1x02_P2.54mm_Vertical
- removed J5: Conn_01x03_Pin, Connector_PinHeader_2.54mm:PinHeader_1x03_P2.54mm_Vertical
- removed TP1: TestPoint, TestPoint:TestPoint_THTPad_D2.0mm_Drill1.0mm
- removed U1: TPS7A0533PDBV, Package_TO_SOT_SMD:SOT-23-5
- added C22: 0.1U, Capacitor_SMD:C_0805_2012Metric_Pad1.18x1.45mm_HandSolder, F.Cu at (70.1, 81.5)
- added C23: 0.1U, Capacitor_SMD:C_0805_2012Metric_Pad1.18x1.45mm_HandSolder, F.Cu at (74.1, 82.1)
- added C24: 10U, Capacitor_SMD:C_1206_3216Metric_Pad1.33x1.80mm_HandSolder, F.Cu at (80.4, 99.2)
- added C25: 0.1U, Capacitor_SMD:C_0805_2012Metric_Pad1.18x1.45mm_HandSolder, F.Cu at (73.2, 98.4)
- added C26: 10u, Capacitor_THT:C_Radial_D6.3mm_H5.0mm_P2.50mm, F.Cu at (87.0, 108.0)
- added C27: 1.3n, Capacitor_SMD:C_0805_2012Metric_Pad1.18x1.45mm_HandSolder, F.Cu at (101.5, 74.4)
- added C28: 560p, Capacitor_SMD:C_0805_2012Metric_Pad1.18x1.45mm_HandSolder, F.Cu at (105.5, 74.4)
- added C29: 1.3n, Capacitor_SMD:C_0805_2012Metric_Pad1.18x1.45mm_HandSolder, F.Cu at (101.5, 78.0)
- added C30: 560p, Capacitor_SMD:C_0805_2012Metric_Pad1.18x1.45mm_HandSolder, F.Cu at (105.5, 78.0)
- added C31: 1.3n, Capacitor_SMD:C_0805_2012Metric_Pad1.18x1.45mm_HandSolder, F.Cu at (101.5, 88.4)
- added C32: 560p, Capacitor_SMD:C_0805_2012Metric_Pad1.18x1.45mm_HandSolder, F.Cu at (105.5, 88.4)
- added C33: 1.3n, Capacitor_SMD:C_0805_2012Metric_Pad1.18x1.45mm_HandSolder, F.Cu at (101.5, 91.9)
- added C34: 560p, Capacitor_SMD:C_0805_2012Metric_Pad1.18x1.45mm_HandSolder, F.Cu at (105.5, 91.9)
- added C35: 1.3n, Capacitor_SMD:C_0805_2012Metric_Pad1.18x1.45mm_HandSolder, F.Cu at (105.5, 102.3)
- added C36: 560p, Capacitor_SMD:C_0805_2012Metric_Pad1.18x1.45mm_HandSolder, F.Cu at (101.5, 102.3)
- added C37: 560p, Capacitor_SMD:C_0805_2012Metric_Pad1.18x1.45mm_HandSolder, F.Cu at (101.5, 105.8)
- added C38: 1.3n, Capacitor_SMD:C_0805_2012Metric_Pad1.18x1.45mm_HandSolder, F.Cu at (105.5, 105.8)
- added C39: 0.1U, Capacitor_SMD:C_0805_2012Metric_Pad1.18x1.45mm_HandSolder, F.Cu at (97.2, 81.8)
- added C40: 0.1U, Capacitor_SMD:C_0805_2012Metric_Pad1.18x1.45mm_HandSolder, F.Cu at (97.4, 95.8)
- added C41: 0.1U, Capacitor_SMD:C_0805_2012Metric_Pad1.18x1.45mm_HandSolder, F.Cu at (97.1, 110.2)
- added C42: 0.1U, Capacitor_SMD:C_0805_2012Metric_Pad1.18x1.45mm_HandSolder, F.Cu at (93.4, 83.4)
- added C43: 0.1U, Capacitor_SMD:C_0805_2012Metric_Pad1.18x1.45mm_HandSolder, F.Cu at (93.7, 97.5)
- added C44: 0.1U, Capacitor_SMD:C_0805_2012Metric_Pad1.18x1.45mm_HandSolder, F.Cu at (94.3, 70.4)
- added R10: 2.33k, Resistor_SMD:R_0805_2012Metric_Pad1.20x1.40mm_HandSolder, F.Cu at (101.4, 84.9)
- added R11: 5.1k, Resistor_SMD:R_0805_2012Metric_Pad1.20x1.40mm_HandSolder, F.Cu at (105.4, 84.9)
- added R12: 47R, Resistor_SMD:R_0805_2012Metric_Pad1.20x1.40mm_HandSolder, F.Cu at (108.6, 86.7)
- added R13: 2.33k, Resistor_SMD:R_0805_2012Metric_Pad1.20x1.40mm_HandSolder, F.Cu at (101.4, 95.3)
- added R14: 5.1k, Resistor_SMD:R_0805_2012Metric_Pad1.20x1.40mm_HandSolder, F.Cu at (105.4, 95.3)
- added R15: 47R, Resistor_SMD:R_0805_2012Metric_Pad1.20x1.40mm_HandSolder, F.Cu at (108.6, 93.6)
- added R16: 2.33k, Resistor_SMD:R_0805_2012Metric_Pad1.20x1.40mm_HandSolder, F.Cu at (101.4, 98.8)
- added R17: 5.1k, Resistor_SMD:R_0805_2012Metric_Pad1.20x1.40mm_HandSolder, F.Cu at (105.4, 98.8)
- added R18: 2.33k, Resistor_SMD:R_0805_2012Metric_Pad1.20x1.40mm_HandSolder, F.Cu at (105.4, 109.3)
- added R19: 5.1k, Resistor_SMD:R_0805_2012Metric_Pad1.20x1.40mm_HandSolder, F.Cu at (101.4, 109.3)
- added R20: 47R, Resistor_SMD:R_0805_2012Metric_Pad1.20x1.40mm_HandSolder, F.Cu at (108.6, 100.5)
- added R21: 47R, Resistor_SMD:R_0805_2012Metric_Pad1.20x1.40mm_HandSolder, F.Cu at (108.6, 107.4)
- added R9: 47R, Resistor_SMD:R_0805_2012Metric_Pad1.20x1.40mm_HandSolder, F.Cu at (108.6, 72.9)
- added U3: OPA2156xD, Package_SO:SOIC-8_3.9x4.9mm_P1.27mm, F.Cu at (95.4, 75.5)
- added U4: OPA2156xD, Package_SO:SOIC-8_3.9x4.9mm_P1.27mm, F.Cu at (95.4, 89.7)
- added U5: OPA2156xD, Package_SO:SOIC-8_3.9x4.9mm_P1.27mm, F.Cu at (95.4, 103.9)
- C10, C12: value 2.2u 25V -> 10u; footprint Capacitor_SMD:C_1206_3216Metric_Pad1.33x1.80mm_HandSolder -> Capacitor_THT:C_Radial_D6.3mm_H5.0mm_P2.50mm
- C2, C3: value 2.2n 50V C0G -> 10u; footprint Capacitor_SMD:C_0805_2012Metric_Pad1.18x1.45mm_HandSolder -> Capacitor_THT:C_Radial_D6.3mm_H5.0mm_P2.50mm
- C20: value 0.1U -> 10U; footprint Capacitor_SMD:C_0805_2012Metric_Pad1.18x1.45mm_HandSolder -> Capacitor_SMD:C_1206_3216Metric_Pad1.33x1.80mm_HandSolder
- C4, C5: value 22U-47U -> 220u; footprint Capacitor_SMD:C_1206_3216Metric_Pad1.33x1.80mm_HandSolder -> Capacitor_THT:CP_Radial_D6.3mm_P2.50mm
- C9: value 10U -> 10u; footprint Capacitor_SMD:C_1206_3216Metric_Pad1.33x1.80mm_HandSolder -> Capacitor_THT:C_Radial_D6.3mm_H5.0mm_P2.50mm
- J10, J14, J15: value Conn_01x02_Pin -> Conn_01x02; footprint Connector_PinHeader_2.54mm:PinHeader_1x02_P2.54mm_Vertical -> TerminalBlock_Phoenix:TerminalBlock_Phoenix_PT-1,5-2-3.5-H_1x02_P3.50mm_Horizontal
- J11, J16: value Conn_01x03_Pin -> Conn_01x02; footprint Connector_JST:JST_PH_B3B-PH-K_1x03_P2.00mm_Vertical -> TerminalBlock_Phoenix:TerminalBlock_Phoenix_PT-1,5-2-3.5-H_1x02_P3.50mm_Horizontal
- J18: value Conn_01x04_Pin -> -12V; footprint Connector_JST:JST_PH_B4B-PH-K_1x04_P2.00mm_Vertical -> Connector_JST:JST_PH_B3B-PH-K_1x03_P2.00mm_Vertical
- J4: value Conn_01x03 -> Conn_01x02; footprint TerminalBlock_Phoenix:TerminalBlock_Phoenix_PT-1,5-3-3.5-H_1x03_P3.50mm_Horizontal -> TerminalBlock_Phoenix:TerminalBlock_Phoenix_PT-1,5-2-3.5-H_1x02_P3.50mm_Horizontal
- R4: value 470R TF -> 2.33k
- R5: value 470R TF -> 5.1k
- R6: value 4.7K -> 2.33k
- R7: value 4.7K -> 5.1k
- R8: value 4.7K -> 47R
- TP2, TP3, TP4, TP5: footprint TestPoint:TestPoint_THTPad_D2.0mm_Drill1.0mm -> TestPoint:TestPoint_THTPad_1.5x1.5mm_Drill0.7mm
- U2: value PCM5122PW -> PCM1681PWPR; footprint Package_SO:TSSOP-28_4.4x9.7mm_P0.65mm -> easyeda2kicad:TSSOP-28_L9.7-W4.4-P0.65-LS6.4-BL-EP-3
- moved J18 56.5 mm to (130.6, 95.4), turned to 90 degrees
- moved J11 43.4 mm to (93.5, 63.3), turned to 180 degrees
- moved J15 40.8 mm to (111.3, 63.3), turned to 180 degrees
- moved TP4 40.7 mm to (62.3, 83.9)
- moved J14 40.5 mm to (102.4, 63.3), turned to 180 degrees
- moved J16 39.8 mm to (120.3, 63.3), turned to 180 degrees
- moved R6 38.0 mm to (101.4, 81.4)
- moved J10 35.6 mm to (84.5, 63.3), turned to 180 degrees
- moved R4 35.0 mm to (105.4, 71.0), turned to 0 degrees
- moved TP5 33.7 mm to (117.4, 109.1)
- moved R8 30.4 mm to (108.6, 79.8), turned to -90 degrees
- moved J13 27.9 mm to (78.3, 94.5), turned to 180 degrees
- moved J4 27.8 mm to (75.6, 63.3)
- moved J8 27.6 mm to (130.4, 83.9)
- moved R5 27.1 mm to (101.4, 71.0), turned to 0 degrees
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Connections:
- C10 pad 1: AGND -> CHAN4
- C10 pad 2: Net-(U2-VNEG) -> Net-(C10-Pad2)
- C12 pad 1: Net-(U2-CAPP) -> CHAN5
- C12 pad 2: Net-(U2-CAPM) -> Net-(C12-Pad2)
- C15 pad 1: Net-(U1-EN) -> 5VA
- C16 pad 1: Net-(U1-EN) -> 5VA
- C2 pad 1: AGND -> CHAN1
- C2 pad 2: LEFT_TWEETER -> Net-(C2-Pad2)
- C20 pad 1: GND -> Net-(U2-VCOM)
- C20 pad 2: Net-(U2-LDOO) -> AGND
- C21 pad 1: Net-(U2-LDOO) -> AGND
- C21 pad 2: GND -> 5VA
- C3 pad 1: AGND -> CHAN2
- C3 pad 2: LEFT_WOOFER -> Net-(C3-Pad2)
- C4 pad 1: 3V3A -> 12V
- C5 pad 1: 3V3A -> AGND
- C5 pad 2: AGND -> -12V
- C9 pad 1: 3V3A -> CHAN3
- C9 pad 2: AGND -> Net-(C9-Pad2)
- D3 pad 1: AGND -> -12V
- FB1 pad 2: Net-(U1-EN) -> 5VA
- J10 pad 1: ADDR2 -> AGND
- J10 pad 2: 3V3 -> OUT2
- J11 pad 1: 3V3 -> AGND
- J11 pad 2: GND_IN -> OUT3
- J12 pad 2: GND_IN -> GND
- J14 pad 1: ADDR1 -> AGND
- J14 pad 2: 3V3 -> OUT4
- J15 pad 1: XSMT -> AGND
- J15 pad 2: XSMT_IN -> OUT5
- J16 pad 1: SCL -> AGND
- J16 pad 2: SDA -> OUT6
- J18 pad 1: SCLK -> -12V
- J18 pad 2: BCLK -> ANALOG_GND
- J18 pad 3: LRCLK -> 12V
- J4 pad 1: LEFT_WOOFER -> AGND
- J4 pad 2: AGND -> OUT1
- J8 pad 1: GND -> ANALOG_GND
- R3 pad 1: 3V3A -> 12V
- R4 pad 1: LT_OUT_PRE -> Net-(C2-Pad2)
- R4 pad 2: LEFT_TWEETER -> Net-(C27-Pad1)
- R5 pad 1: LW_OUT_PRE -> Net-(C27-Pad1)
- R5 pad 2: LEFT_WOOFER -> Net-(U3A-+)
- R6 pad 1: GND -> Net-(C3-Pad2)
- R6 pad 2: ADDR2 -> Net-(C29-Pad1)
- R7 pad 1: 3V3 -> Net-(C29-Pad1)
- R7 pad 2: XSMT -> Net-(U3B-+)
- R8 pad 1: GND -> Net-(U3B--)
- R8 pad 2: ADDR1 -> OUT2
- U2 pad 1: 3V3A -> ZR1
- U2 pad 10: AGND -> GND
- U2 pad 11: SDA -> DATA2
- U2 pad 12: SCL -> DATA3
- U2 pad 13: unconnected-(U2-GPIO5/ATT0-Pad13) -> DATA4
- U2 pad 14: unconnected-(U2-GPIO4/MAST-Pad14) -> GND
- U2 pad 15: unconnected-(U2-GPIO3/AGNS-Pad15) -> CHAN8
- U2 pad 16: ADDR2 -> CHAN7
- U2 pad 17: GND -> 5VA
- U2 pad 18: 3V3 -> AGND
- U2 pad 19: unconnected-(U2-GPIO6/FLT-Pad19) -> CHAN6
- U2 pad 2: Net-(U2-CAPP) -> ADDR
- U2 pad 20: SCLK -> CHAN5
- U2 pad 21: BCLK -> CHAN4
- U2 pad 22: DATA -> CHAN3
- U2 pad 23: LRCLK -> 5VA
- U2 pad 24: ADDR1 -> AGND
- U2 pad 25: XSMT -> Net-(U2-VCOM)
- U2 pad 26: Net-(U2-LDOO) -> CHAN2
- U2 pad 27: GND -> CHAN1
- U2 pad 28: 3V3 -> ZR2
- U2 pad 3: AGND -> SCL
- U2 pad 4: Net-(U2-CAPM) -> SDA
- U2 pad 5: Net-(U2-VNEG) -> SCLK
- U2 pad 6: LW_OUT_PRE -> DATA1
- U2 pad 7: LT_OUT_PRE -> BCLK
- U2 pad 8: 3V3A -> LRCLK
- U2 pad 9: AGND -> 3V3
Routing:
- net 3V3: track 156.2 -> 0.00 mm, vias 11 -> 0
- net SCL: track 106.2 -> 0.00 mm, vias 9 -> 0
- net SDA: track 106.2 -> 0.00 mm, vias 11 -> 0
- net 3V3A: track 95.0 -> 0.00 mm, vias 9 -> 0
- net LEFT_WOOFER: track 77.4 -> 0.00 mm, vias 1 -> 0
- net 5V: track 70.3 -> 0.00 mm, vias 5 -> 0
- net LEFT_TWEETER: track 47.5 -> 0.00 mm, vias 1 -> 0
- net AGND: track 39.8 -> 0.00 mm, vias 15 -> 0
- net XSMT: track 37.9 -> 0.00 mm, vias 2 -> 0
- net DATA: track 37.3 -> 0.00 mm, vias 2 -> 0
- net LRCLK: track 34.6 -> 0.00 mm, vias 2 -> 0
- net SCLK: track 33.2 -> 0.00 mm, vias 1 -> 0
- net BCLK: track 33.0 -> 0.00 mm, vias 2 -> 0
- net GND_IN: track 25.8 -> 0.00 mm, vias 1 -> 0
- net ADDR1: track 25.5 -> 0.00 mm, vias 2 -> 0
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- removed copper zone on B.Cu, net AGND
- removed copper zone on F.Cu, net GND
Other:
- board text added: "AGND/ANAG"
- board text added: "ANALOG_PWR"
- board text added: "APWR"
- board text added: "DAC PCM1681 1.0"
- board text added: "DIGITAL_PWR"
- board text added: "I2S1"
- board text added: "OUT1"
- board text added: "OUT2"
- board text added: "OUT3"
- board text added: "OUT4"
- board text added: "OUT5"
- board text added: "OUT6"
- board text removed: "3V3A"
- board text removed: "ADDR1"
- board text removed: "ADDR2"
- board text removed: "AGND/GND"
- board text removed: "AUDIO_OUT"
- board text removed: "CTRL_IN"
- board text removed: "CTRL_OUT"
- board text removed: "DAC PCM5122 1.0"
- board text removed: "GND_IN"
- board text removed: "I2S"
- board text removed: "I2S_DEBUG"
- board text removed: "LT"
- board text removed: "LW"
- board text removed: "LW/GND/LT"
- board text removed: "POWER_IN"
- board text removed: "POWER_OUT"
- board text removed: "XSMT"
