File: pcbs/_final_proto/i2s/1.0/i2s.kicad_pcb (KiCad board)
At the start: 2 copper layers, 75 x 55 mm, 41 parts, among them J1 Conn_01x04_Pin, J10 Conn_01x02, J2 Conn_01x04_Pin, J3 Conn_01x04_Pin, J4 Conn_01x04_Pin, J5 Conn_01x04_Pin, J6 Conn_01x04_Pin, J7 Conn_01x04_Pin, J8 Conn_01x03, J9 Conn_01x02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

Commit message: Working code
Parts:
- C1: renamed from C5; footprint Capacitor_THT:CP_Radial_D6.3mm_P2.50mm -> Capacitor_SMD:CP_Elec_6.3x7.7
- C2: renamed from C1; footprint Capacitor_SMD:C_1206_3216Metric_Pad1.33x1.80mm_HandSolder -> Custom:C_1206_3216Metric_Pad1.33x1.80mm_HandSolder_Duane
- C3: renamed from C2; footprint Capacitor_SMD:C_0805_2012Metric_Pad1.18x1.45mm_HandSolder -> Custom:C_0805_2012Metric_Pad1.18x1.45mm_HandSolder_Duane
- C4: renamed from C3; footprint Capacitor_SMD:C_0805_2012Metric_Pad1.18x1.45mm_HandSolder -> Custom:C_0805_2012Metric_Pad1.18x1.45mm_HandSolder_Duane
- C5: renamed from C4; footprint Capacitor_SMD:C_0805_2012Metric_Pad1.18x1.45mm_HandSolder -> Custom:C_0805_2012Metric_Pad1.18x1.45mm_HandSolder_Duane
- D1, D2, D3, D4, D5: footprint LED_SMD:LED_0805_2012Metric_Pad1.15x1.40mm_HandSolder -> Custom:LED_0805_2012Metric_Pad_HandSolder_Duane
- R1, R10, R11, R12, R13, R14, R2, R3, R4, R7, R8, R9: footprint Resistor_SMD:R_0805_2012Metric_Pad1.20x1.40mm_HandSolder -> Custom:R_0805_2012Metric_Pad1.20x1.40mm_HandSolder_Duane
- R5: renamed from R6; footprint Resistor_SMD:R_0805_2012Metric_Pad1.20x1.40mm_HandSolder -> Custom:R_0805_2012Metric_Pad1.20x1.40mm_HandSolder_Duane
- R6: renamed from R5; footprint Resistor_SMD:R_0805_2012Metric_Pad1.20x1.40mm_HandSolder -> Custom:R_0805_2012Metric_Pad1.20x1.40mm_HandSolder_Duane
- moved C1 13.3 mm to (156.9, 86.4), turned to -90 degrees
- moved R6 9.63 mm to (158.1, 101.0)
- moved D1 9.63 mm to (158.1, 97.2)
- moved C5 9.11 mm to (124.6, 94.5)
- moved U2 9.11 mm to (143.2, 87.2)
- moved C2 9.11 mm to (136.2, 90.3)
- moved U1 9.11 mm to (122.4, 87.2)
- moved C3 9.11 mm to (140.3, 92.8)
- moved C4 4.87 mm to (107.5, 94.7)
- moved R1 4.87 mm to (103.4, 80.4)
- moved U3 4.87 mm to (105.1, 87.9)
- renumbered U2 to U1, U3 to U2, U1 to U3
Connections:
- R1 pad 1: GND -> 3V3
Routing:
- net 3V3: track 142.2 -> 179.5 mm, vias 10 -> 16
- net I2S_LRCLK: track 39.5 -> 74.3 mm, vias 0 -> 4
- net EN4: track 109.5 -> 76.8 mm, vias 6 -> 3
- net I2S_BCLK: track 45.5 -> 68.7 mm, vias 6 -> 8
- net EN2: track 94.3 -> 71.3 mm, vias 8 -> 3
- net Net-(U3-1Y): track 9.60 -> 27.9 mm, vias 2 -> 4
- net I2S_MCLK: track 50.3 -> 65.6 mm, vias 6 -> 10
- net I2S_LRCLK_4: track 22.7 -> 36.3 mm, vias 1 -> 3
- net I2S_BCLK_3: track 22.6 -> 34.5 mm, vias 1 -> 3
- net I2S_DATA_3: track 19.2 -> 30.2 mm, vias 1 -> 3
- net I2S_LRCLK_2: track 21.5 -> 32.5 mm
- net I2S_DATA_4: track 27.0 -> 37.7 mm, vias 1 -> 3
- net I2S_BCLK_2: track 19.5 -> 29.5 mm
- net I2S_DATA_2: track 25.0 -> 34.5 mm
- net I2S_BCLK_4: track 20.1 -> 29.5 mm
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Other:
- board text added: "I2S 1.1"
- board text removed: "I2S 1.0"
