File: pcbs/_final_proto/i2s/1.0/i2s.kicad_sch (KiCad schematic)
At the start: 41 parts, among them J1 Conn_01x04_Pin, J10 Conn_01x02, J2 Conn_01x04_Pin, J3 Conn_01x04_Pin, J4 Conn_01x04_Pin, J5 Conn_01x04_Pin, J6 Conn_01x04_Pin, J7 Conn_01x04_Pin, J8 Conn_01x03, J9 Conn_01x02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

Commit message: Working code
Parts:
- C1: renamed from C5; footprint Capacitor_THT:CP_Radial_D6.3mm_P2.50mm -> Capacitor_SMD:CP_Elec_6.3x7.7
- C2: renamed from C1; footprint Capacitor_SMD:C_1206_3216Metric_Pad1.33x1.80mm_HandSolder -> Custom:C_1206_3216Metric_Pad1.33x1.80mm_HandSolder_Duane
- C3: renamed from C2; footprint Capacitor_SMD:C_0805_2012Metric_Pad1.18x1.45mm_HandSolder -> Custom:C_0805_2012Metric_Pad1.18x1.45mm_HandSolder_Duane
- C4: renamed from C3; footprint Capacitor_SMD:C_0805_2012Metric_Pad1.18x1.45mm_HandSolder -> Custom:C_0805_2012Metric_Pad1.18x1.45mm_HandSolder_Duane
- C5: renamed from C4; footprint Capacitor_SMD:C_0805_2012Metric_Pad1.18x1.45mm_HandSolder -> Custom:C_0805_2012Metric_Pad1.18x1.45mm_HandSolder_Duane
- D1, D2, D3, D4, D5: footprint LED_SMD:LED_0805_2012Metric_Pad1.15x1.40mm_HandSolder -> Custom:LED_0805_2012Metric_Pad_HandSolder_Duane
- R1, R10, R11, R12, R13, R14, R2, R3, R4, R7, R8, R9: footprint Resistor_SMD:R_0805_2012Metric_Pad1.20x1.40mm_HandSolder -> Custom:R_0805_2012Metric_Pad1.20x1.40mm_HandSolder_Duane
- R5: renamed from R6; footprint Resistor_SMD:R_0805_2012Metric_Pad1.20x1.40mm_HandSolder -> Custom:R_0805_2012Metric_Pad1.20x1.40mm_HandSolder_Duane
- R6: renamed from R5; footprint Resistor_SMD:R_0805_2012Metric_Pad1.20x1.40mm_HandSolder -> Custom:R_0805_2012Metric_Pad1.20x1.40mm_HandSolder_Duane
- renumbered U2 to U1, U3 to U2, U1 to U3
Connections:
- net 3V3: now also R1.1
- net GND: no longer R1.1
