File: pcbs/_final_proto/lift/1.0/lift.kicad_sch (KiCad schematic)
At the start: 12 parts, among them J1 Conn_01x03_Pin, J2 Conn_01x03_Pin, J3 Conn_01x02_Male, J4 Conn_01x02, J5 Conn_01x02_Male

Commit message: Working code
Parts:
- C1: value 100n X2 250V -> 100n X2 (Switch to Y2) 250V
Changed lines of the file:
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@@
 			)
 		)
-		(property "Value" "100n X2 250V"
+		(property "Value" "100n X2 (Switch to Y2) 250V"
 			(at 39.116 71.374 90)
 			(effects
