File: pcbs/plate-amp/2.0/plate-amp.kicad_sch (KiCad schematic)
At the start: 104 parts, among them J1 Conn_01x02_Pin, J2 Conn_01x02_Pin, J3 Conn_01x02_Pin, J4 Conn_01x02_Pin, J5 Conn_01x02_Pin, J6 Conn_01x02_Pin, J7 Conn_01x02_Pin, U1 AP64351SP-13, U4 LM317_SOT-223, U5 TPA3255DDV, U6 OPA1602, U7 OPA1602

Commit message: Working code
Parts:
- added C52, C53: 10u Nichicon 25V, Capacitor_THT:CP_Radial_D5.0mm_P2.50mm, symbol Device:C_Small
- added J5: Conn_01x02_Pin, Connector_PinHeader_2.54mm:PinHeader_1x02_P2.54mm_Vertical, symbol Connector:Conn_01x02_Pin
- added J6: Conn_01x02_Pin, Connector_JST:JST_PH_B2B-PH-K_1x02_P2.00mm_Vertical, symbol Connector:Conn_01x02_Pin
- added R29: 24k, Capacitor_SMD:C_0603_1608Metric_Pad1.08x0.95mm_HandSolder, symbol Device:R_Small
- added R30, R31, R33: 10k, Capacitor_SMD:C_0603_1608Metric_Pad1.08x0.95mm_HandSolder, symbol Device:R_Small
- added TP2: TestPoint, TestPoint:TestPoint_THTPad_2.5x2.5mm_Drill1.2mm, symbol Connector:TestPoint
- added U8: OPA2134, Package_SO:SOIC-8_3.9x4.9mm_P1.27mm, symbol Amplifier_Operational:OPA2134
- renumbered C4 to C3, C39 to C35, C40 to C36, C35 to C37, C36 to C38, C37 to C39, C5 to C4, C38 to C40, C49 to C48, C48 to C49, C3 to C5, J3 to J2, J2 to J3, J5 to J7, J6 to J8, J7 to J9, R29 to R32
Connections:
- net 4.75V: now also R33.1, U8.3 (+); no longer C51.1, U6.3 (+), U6.5 (+), U7.3 (+), U7.5 (+)
- net 9.5V: now also U8.8 (V+)
- net FAULT: now also J6.2 (Pin_2)
- net GND: now also R29.2, R30.2, R31.2, U8.4 (V-)
- net LEFT_IN: now also C52.2; no longer R24.2
- net RESET: now also J5.1 (Pin_1), J6.1 (Pin_1)
- net RIGHT_IN: now also C53.2; no longer R26.2
- new net: C52.1, R24.2, R30.1
- new net: R29.1, R33.2, U8.5 (+)
- new net: C53.1, R26.2, R31.1
- new net 3.3V: J5.2 (Pin_2), U8.6 (-), U8.7
- new net 4.75VBUF: C51.1, TP2.1, U6.3 (+), U6.5 (+), U7.3 (+), U7.5 (+), U8.1, U8.2 (-)
Other:
- moved on the sheet: C51
